File: 2-speaker-subwoofer/amplifier-pcb/amplifier-pcb.sch (KiCad schematic (older format))
At the start: 16 parts, among them J3 CUI_PD-30, U5 LM7812_TO220

Commit message: added the majority of the components
Parts:
- added C1, C100, C101, C13, C16, C31, C44, C45: 1000pF 10% 100V, symbol Device:C
- added C10, C29: 100000pF 10% 100V, symbol Device:C
- added C103, C20, C3, C51: 1uF 50V, symbol Device:CP1
- added C104, C21, C47: 47uF 16V, symbol Device:CP1
- added C105, C106: 100pF, symbol Device:C
- added C11, C30, C46: 33000pF 5% 100V, symbol Device:C
- added C12, C22, C24, C4: 220nF, symbol Device:C
- added C14, C25, C55, C6: 10000pF 5% 100V, symbol Device:C
- added C18, C2, C56, C59, C60: 2.2uF 50V, symbol Device:CP1
- added C23, C39, C7: 10uF 25V, symbol Device:CP1
- added C26, C9: 0.33uF, symbol Device:C
- added C38, C49, C64: 0.1uF 50V, symbol Device:CP1
- added C41, C43: 470uF 16V, symbol Device:CP1
- added C48: 100uF 16V, symbol Device:CP1
- added C50, C54: 220000pF 5% 100V, symbol Device:C
- added C53, C61, C67, C68, C69: 4.7uF 50V, symbol Device:CP1
- added C63: 0.47uF 50V, symbol Device:CP1
- added D1, D2: D, symbol Device:D
- added J4: RIGHT SPEAKER, symbol Connector_Generic_Shielded:Conn_01x09_Shielded
- added J5: SUB OUT, symbol Connector_Generic:Conn_01x02
- added J6: Conn_01x03, symbol Connector_Generic:Conn_01x03
- added Q3: 2SA1015, Package_TO_SOT_THT:TO-92_Inline, symbol Transistor_BJT:2SA1015
- added Q4: 2SK192A, symbol Device:Q_NMOS_DSG
- added Q5, Q6: 2SC1815, Package_TO_SOT_THT:TO-92_Inline, symbol Transistor_BJT:2SC1815
- added R1, R2, R3: 47kΩ 5%, symbol Device:R
- added R11, R30: 1k8Ω 5%, symbol Device:R
- added R14, R31: 680Ω 5%, symbol Device:R
- added R15, R32, R64, R69: 390Ω 5%, symbol Device:R
- added R17, R35, R56: 3k3Ω 5%, symbol Device:R
- added R18, R4, R48, R63, R68, R79, R80: 22kΩ 5%, symbol Device:R
- added R19, R25: 27kΩ 5%, symbol Device:R
- added R22, R23, R24, R26, R27, R5, R52, R55, R62, R8: 10kΩ 5%, symbol Device:R
- added R38: 470Ω 5%, symbol Device:R
- added R41, R76: 1kΩ 5%, symbol Device:R
- added R43, R44: 560Ω 5%, symbol Device:R
- added R45: 39kΩ 5%, symbol Device:R
- added R53: 12kΩ 5%, symbol Device:R
- added R54: 100kΩ 5%, symbol Device:R
- added R67, R70: 2k2Ω 5%, symbol Device:R
- added R77: 18kΩ 5%, symbol Device:R
- added R78: 2k7Ω 5%, symbol Device:R
- added U1, U2, U6: MC4558CN, symbol Amplifier_Operational:RC4558
- added U10, U9: STA7360, SW-ST:MultiWatt11_(Vertical), symbol SW-ST:STA7360
- added U?: LM1036, symbol SW-Texas:LM1036
- C36, C37, C?: Characteristics (none) -> electrolytic; Manufacturer (none) -> SAMXON
Connections:
- net +12V: no longer D7.2 (A), U5.3 (VO)
- net GND: now also U10.6 (P-GND), U9.6 (P-GND)
- net UNREG_DC_IN renamed +VDC
- net +VDC: now also U10.9 (+Vs), U9.9 (+Vs)
- new net: D7.2 (A), U5.3 (VO)
Other:
- note added: "2A102K = 1000pF 10% 100V\n2A103J = 10000pF 5% 100V\n2A104K = 100000pF 10% 100V\n2A333J = 33000pF 5% 100V\n2A224J = 220000pF 5% 100V"
- note added: "Non Standard 9 pin mini DIN"
- moved on the sheet: C37, D7, JP1, R34, R37

Commit message: lots of updates on schematic
got controller and preamps done, working on amps and discrete transistors
Parts:
- added JP11, JP13, JP14, JP15, JP16, JP18, JP19, JP2, JP24, JP25, JP26, JP3, JP4, JP5, JP8: Jumper, symbol Device:Jumper
- added R20: 10kΩ 5%, symbol Device:R
- added R75: 1kΩ 5%, symbol Device:R
- J6: value Conn_01x03 -> AUDIO_IN
Connections:
- net +12V: now also C14.1, JP1.2, Q3.2 (C), R34.1, R38.2, U1.8 (V+), U2.8 (V+), U?.11 (VCC), JP13.1
- net GND: now also C100.2, C101.2, C105.2, C106.2, C12.2, C14.2, C21.2, C22.2, C23.2, C24.1, C25.2, C26.2, C4.2, C44.2, C45.2, C6.2, C67.2, C68.2, C7.2, C9.2, J4.SH (Shield), J6.3 (Pin_3), R14.2, R15.2, R25.1, R27.2, R31.2, R32.2, R70.1, U1.4 (V-), U2.4 (V-), U6.4 (V-), U?.10 (GND), U?.20 (GND), JP2.1
- net at C37.1, R34.2: now also R18.2, R37.2, R4.2, JP24.1; no longer R37.1
- net at C37.2: now also J4.5 (Pin_5), R26.1, R37.1, JP2.2; no longer R37.2
- net OUT1: now reaches U9.1 (IN1(+))
- net OUT1: now also JP15.2
- net OUT2: now reaches U9.5 (IN2(+))
- net OUT2: now also JP11.2
- net at R70.2: now also Q5.1 (E), R69.1
- net at R15.1: now also C11.1
- net at R48.1: now also R63.1, R68.1, JP24.2
- net at R48.2: now also C59.1, U6.3 (+)
- net at R63.2: now also JP18.2
- net at R68.2: now also C64.1, Q5.3 (B)
- net at R35.1: now also C30.1, C31.2, R30.1, U2.6 (-)
- net at R35.2: now also C68.1
- net at R17.1: now also C11.2, C13.1, R11.1, U2.2 (-)
- net at R17.2: now also C67.1
- net at R43.1: now also C38.2
- net at R43.2: now also C44.1, JP11.1
- net at R44.1: now also C49.2
- net at R44.2: now also C45.1, JP15.1
- net at R38.1: now also Q3.3 (B)
- net at R30.2: now also C31.1, U2.7, JP26.1
- net at R31.1: now also C29.2
- net at R14.1: now also C10.2
- net at R32.1: now also C30.2
- net at R11.2: now also C13.2, U2.1, JP25.1
- net at R76.1: now also C106.1, U?.8 (OUT1)
- net OUT1_PRE: now reaches R76.2
- net OUT1_PRE: now also C100.1, C29.1, U2.5 (+)
- net at R1.1: now also JP3.2
- net at R1.2: now also C4.1, U?.14 (Bass_Cnt)
- net at R3.1: now also JP4.2
- net at R3.2: now also C12.1, U?.12 (Volume_Cnt)
- net at R2.1: now also C22.1, U?.4 (Treble_Cnt)
- net at R2.2: now also JP14.2
- net at R19.1: now also C24.2, R25.2, U?.9 (Balance_Cnt)
- net at R19.2: now also U?.17 (Zener_Voltage), U?.7 (Loudness_Comp_Cnt), JP8.2
- net at R18.1: now also U1.5 (+)
- net at R4.1: now also U1.3 (+)
- net at R24.1: now also C16.1, U1.7, R20.2
- net at R24.2: now also C20.2
- net at R8.1: now also C1.1, R5.1, U1.1
- net at R8.2: now also C3.2
- net at R5.2: now also C1.2, C2.1, U1.2 (-)
- net at R22.1: now also C2.2
- net at R22.2: now also J6.1 (Pin_1), R26.2
- net at R23.1: now also C18.2
- net at R23.2: now also J6.2 (Pin_2), R27.1
- net at C18.1: now also C16.2, U1.6 (-), R20.1
- net IN2: now reaches C3.1
- net IN2: now also U?.19 (IN2)
- net IN1: now reaches C20.1
- net IN1: now also U?.2 (IN1)
- net at C21.1: now also U?.1 (Int_Supply_Decouple)
- net at C23.1: now also U?.5 (AC_Bypass_1)
- net at C7.1: now also U?.16 (AC_Bypass_2)
- net at C64.2: now also C59.2
- net at C38.1: now also JP25.2
- net at C49.1: now also JP26.2
- net at Q6.2 (C): now also JP19.2
- net at Q5.2 (C): now also U6.8 (V+), JP13.2, JP19.1
- net OUT2_PRE: now reaches U2.3 (+)
- net OUT2_PRE: now also C10.1, C101.1, R75.2
- net at C25.1: now also U?.3 (Treble_CAP_1)
- net at C6.1: now also U?.18 (Treble_CAP_2)
- net at C26.1: now also U?.6 (Bass_CAP_1)
- net at C9.1: now also U?.15 (Bass_CAP_2)
- net at C105.1: now also U?.13 (OUt2), JP16.1
- net PIN3: now reaches J4.3 (Pin_3)
- net PIN3: now also JP5.2
- net Volume_Cnt: now reaches J4.7 (Pin_7)
- net Volume_Cnt: now also JP4.1
- net Treble_Cnt: now reaches J4.8 (Pin_8)
- net Treble_Cnt: now also JP14.1
- net Bass_Cnt: now reaches J4.9 (Pin_9)
- net Bass_Cnt: now also JP3.1
- new net: JP5.1, JP8.1
- new net: JP16.2, R75.1
Other:
- note added: "MINI DIN 9\npin numbering\n 1 - 2 - 3\n4 - 5 - 6 -7\n 8 - 9"
- note added: "PCB layout\n\n 4 - 8 - 9 - 7\n5 - 1 - 2 - 6 - 3"
- note added: "pin 1 = white\npin 2 = red\npin 3 = black"
- moved on the sheet: C1, C10, C100, C101, C103, C104, C105, C106, C11, C12, C13, C14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

Commit message: Finished initial pass on schematic
Parts:
- added JP17, JP21, JP22, JP23, JP6, JP7: Jumper, symbol Device:Jumper
- added R74: 3k3Ω 5%, symbol Device:R
- gave numbers to parts that had none: 1
Connections:
- net +12V: now also Q3.1 (E); no longer Q3.2 (C)
- net GND: now also C50.2, C54.2, C69.2, R55.1, R67.2, JP17.1; no longer C44.2, C45.2, R70.1, U6.4 (V-)
- net at U9.10 (OUT1): now also C43.1
- net STANDBY: now reaches U9.11 (STAND-BY)
- net STANDBY: now also U10.11 (STAND-BY), JP22.1
- net GNDS: now reaches U9.3 (S-GND)
- net GNDS: now also C103.2, C104.2, C39.2, C44.2, C45.2, C46.1, C47.2, R62.2, R70.1, R80.1, U6.4 (V-), JP17.2, JP21.2
- net at U9.4 (OUT_BRIDGE): now also C41.1, U9.8 (OUT2)
- net at U9.7 (SVR): now also C47.1
- net at U10.1 (IN1(+)): now also C46.2, R74.1
- net SUB-OUT-BRIDGE: now reaches U10.10 (OUT1)
- net SUB-OUT-BRIDGE: now also J5.1 (Pin_1), R45.1, U10.4 (OUT_BRIDGE)
- net at U10.3 (S-GND): now also JP21.1
- net at U10.5 (IN2(+)): now also C103.1
- net at U10.7 (SVR): now also C104.1
- net SUB-OUT-AMP: now reaches U10.8 (OUT2)
- net SUB-OUT-AMP: now also JP23.1
- net at R45.2: now also C48.1
- net at D1.1 (K): now also C53.1, R54.1
- net at D1.2 (A): now also C48.2, D2.1 (K), R55.2
- net at D2.2 (A): now also C53.2, Q4.3 (G), R54.2
- net at R64.1: now also C61.1, C63.2
- net at R64.2: now also Q6.1 (E), R67.1
- net at R53.1: now also C50.1, R52.2
- net at R53.2: now also C54.1, U6.5 (+)
- net at R78.1: now also R77.2, U6.6 (-)
- net at R78.2: now also C69.1
- net at R77.1: now also C51.1, U6.7
- net at R52.1: now also C55.2, R56.2, U6.1
- net at R62.1: now also C56.2, Q4.1 (D)
- net at R69.2: now also C59.2, C64.2
- net at C59.1, R48.2, U6.3 (+): now also C60.1
- net at R79.1: now also C39.1, R80.2, JP22.2
- net at R79.2: now also Q3.2 (C)
- net at R56.1: now also C55.1, C56.1, U6.2 (-)
- net at Q3.3 (B), R38.1: now also JP7.1
- net at R41.1: now also JP6.1
- net at R41.2: now also JP7.2
- net at C63.1: now also JP18.1, Q6.3 (B)
- net at C61.2: now also Q4.2 (S)
- net at C51.2: now also R74.2
- net PIN4: now reaches C60.2
- net PIN4: now also J4.4 (Pin_4)
- net OUT2_AMP: now reaches C41.2
- net OUT2_AMP: now also J4.1 (Pin_1)
- net OUT1_AMP: now reaches C43.2
- net OUT1_AMP: now also J4.2 (Pin_2)
- net at J5.2 (Pin_2): now also JP23.2
- net PIN6: now reaches J4.6 (Pin_6)
- net PIN6: now also JP6.2
- no-connect marks 1 -> 3
Other:
- note added: "GND and GNDS are equivalent,\nUsing different symbols due to the jumpers"
- note added: "pin1 = black\npin2 = red"
- moved on the sheet: C103, C104, C39, C41, C43, C46, C47, C48, C50, C51, C53, C54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

Commit message: adding diode part numbers
Parts:
- D1, D2: value D -> 1N4148
- Q4: Manufacturer (none) -> Toshiba; Package ID (none) -> 2-4E1D Toshiba
Changed lines of the file:
@@
 P 4850 14350
 F 0 "D1" H 4850 14150 50  0000 C CNN
-F 1 "D" H 4850 14250 50  0000 C CNN
+F 1 "1N4148" H 4850 14250 50  0000 C CNN
 F 2 "" H 4850 14350 50  0001 C CNN
 F 3 "~" H 4850 14350 50  0001 C CNN
@@
 P 5750 14100
 F 0 "D2" H 5750 13884 50  0000 C CNN
-F 1 "D" H 5750 13975 50  0000 C CNN
+F 1 "1N4148" H 5750 13975 50  0000 C CNN
 F 2 "" H 5750 14100 50  0001 C CNN
 F 3 "~" H 5750 14100 50  0001 C CNN
@@
 F 2 "" H 7200 14750 50  0001 C CNN
 F 3 "~" H 7000 14650 50  0001 C CNN
+F 4 "Toshiba" H 7000 14650 50  0001 C CNN "Manufacturer"
+F 5 "2-4E1D Toshiba" H 7000 14650 50  0001 C CNN "Package ID"
 	1    7000 14650
 	1    0    0    -1

Commit message: Updated pinout info
added more notes, fixed net labels and shrunk page size
Connections:
- net S_GND: now reaches C37.2, J4.5 (Pin_5), JP2.2, R26.1, R37.1
- net IN1 renamed LEFT_IN
- net IN2 renamed RIGHT_IN
- net OUT1 renamed LEFT
- net OUT1_AMP renamed L_SPK
- net OUT1_PRE renamed LEFT_PRE
- net OUT2 renamed RIGHT
- net OUT2_AMP renamed R_SPK
- net OUT2_PRE renamed RIGHT_PRE
- net PIN3 renamed ZENER_VREF
- net PIN4 renamed SUB_RETURN
- net PIN6 renamed PWR_ON
Other:
- note added: "Female to Male pin # \ncross reference\n1 = 3\n2 = 2\n3 = 1\n4 = 7\n5 = 6\n6 = 5\n7 = 4\n8 = 9\n9 = 8"
- note added: "MINI DIN 9\npin numbering\nlooking into the \nfemale board \nconnector\n 1 - 2 - 3\n4 - 5 - 6 -7\n 8 - 9"
- note added: "OUT1 = L\nOUT2 = R"
- note added: "PWR_ON is signal\nfrom right speaker\nto turn power on"
- note added: "wire colors to mini din male pins\nnumbered looking into the connector\non the cable\n 1 - 2 - 3\n4 - 5 - 6 - 7\n 8 - 9\n\nblack = shield\nwhite = 3\ngrey = 2\nbrown = 8\npurple = 1\nblue = 7\ngreen = 6\nyellow = 5\norange = 4\nred = 9"
- note removed: "MINI DIN 9\npin numbering\n 1 - 2 - 3\n4 - 5 - 6 -7\n 8 - 9"
- moved on the sheet: C10, C100, C101, C105, C106, C11, C12, C13, C21, C22, C23, C24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

Commit message: Fixed missing reference designator and added footprint info for more components
Parts:
- D3, D4, D5, D6, D7: value D -> 6A2; Characteristics (none) -> 200V Peak Reverse Voltage, 140VRMS max, 200V max DC blockin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; Description (none) -> power diode
- U1, U2, U6: footprint (none) -> Package_DIP:DIP-8_W7.62mm
- U3: renamed from U?; footprint (none) -> Package_DIP:DIP-20_W7.62mm
Changed lines of the file:
@@
 P 5750 10550
 F 0 "D5" H 5750 10650 50  0000 C CNN
-F 1 "D" H 5750 10450 50  0000 C CNN
+F 1 "6A2" H 5750 10450 50  0000 C CNN
 F 2 "" H 5750 10550 50  0001 C CNN
 F 3 "~" H 5750 10550 50  0001 C CNN
+F 4 "200V Peak Reverse Voltage, 140VRMS max, 200V max DC blocking voltage, 6A Max Avg forward rectified current, peak foward surge current = 400A 8.3ms single half sine wave, max instantaneous forward voltage @6A DC = 0.9V, max DC reverse current @rating blocking voltage, 10uA@+25C, 100uA@+100C" H 5750 10550 50  0001 C CNN "Characteristics"
+F 5 "power diode" H 5750 10550 50  0001 C CNN "Description"
 	1    5750 10550
 	-1   0    0    1
@@
 P 5750 10800
 F 0 "D3" H 5750 10900 50  0000 C CNN
-F 1 "D" H 5750 10700 50  0000 C CNN
+F 1 "6A2" H 5750 10700 50  0000 C CNN
 F 2 "" H 5750 10800 50  0001 C CNN
 F 3 "~" H 5750 10800 50  0001 C CNN
+F 4 "200V Peak Reverse Voltage, 140VRMS max, 200V max DC blocking voltage, 6A Max Avg forward rectified current, peak foward surge current = 400A 8.3ms single half sine wave, max instantaneous forward voltage @6A DC = 0.9V, max DC reverse current @rating blocking voltage, 10uA@+25C, 100uA@+100C" H 5750 10800 50  0001 C CNN "Characteristics"
+F 5 "power diode" H 5750 10800 50  0001 C CNN "Description"
 	1    5750 10800
 	1    0    0    1
@@
 P 5750 10300
 F 0 "D4" H 5750 10400 50  0000 C CNN
-F 1 "D" H 5750 10200 50  0000 C CNN
+F 1 "6A2" H 5750 10200 50  0000 C CNN
 F 2 "" H 5750 10300 50  0001 C CNN
 F 3 "~" H 5750 10300 50  0001 C CNN
+F 4 "200V Peak Reverse Voltage, 140VRMS max, 200V max DC blocking voltage, 6A Max Avg forward rectified current, peak foward surge current = 400A 8.3ms single half sine wave, max instantaneous forward voltage @6A DC = 0.9V, max DC reverse current @rating blocking voltage, 10uA@+25C, 100uA@+100C" H 5750 10300 50  0001 C CNN "Characteristics"
+F 5 "power diode" H 5750 10300 50  0001 C CNN "Description"
 	1    5750 10300
 	1    0    0    1
@@
 P 5300 9350
 F 0 "D7" H 5300 9134 50  0000 C CNN
-F 1 "D" H 5300 9225 50  0000 C CNN
+F 1 "6A2" H 5300 9225 50  0000 C CNN
 F 2 "" H 5300 9350 50  0001 C CNN
 F 3 "~" H 5300 9350 50  0001 C CNN
+F 4 "200V Peak Reverse Voltage, 140VRMS max, 200V max DC blocking voltage, 6A Max Avg forward rectified current, peak foward surge current = 400A 8.3ms single half sine wave, max instantaneous forward voltage @6A DC = 0.9V, max DC reverse current @rating blocking voltage, 10uA@+25C, 100uA@+100C" H 5300 9350 50  0001 C CNN "Characteristics"
+F 5 "power diode" H 5300 9350 50  0001 C CNN "Description"
 	1    5300 9350
 	-1   0    0    1
@@
 P 5750 10050
 F 0 "D6" H 5750 10150 50  0000 C CNN
-F 1 "D" H 5750 9950 50  0000 C CNN
+F 1 "6A2" H 5750 9950 50  0000 C CNN
 F 2 "" H 5750 10050 50  0001 C CNN
 F 3 "~" H 5750 10050 50  0001 C CNN
+F 4 "200V Peak Reverse Voltage, 140VRMS max, 200V max DC blocking voltage, 6A Max Avg forward rectified current, peak foward surge current = 400A 8.3ms single half sine wave, max instantaneous forward voltage @6A DC = 0.9V, max DC reverse current @rating blocking voltage, 10uA@+25C, 100uA@+100C" H 5750 10050 50  0001 C CNN "Characteristics"
+F 5 "power diode" H 5750 10050 50  0001 C CNN "Description"
 	1    5750 10050
 	-1   0    0    1
@@
 F 0 "U6" H 8850 12850 50  0000 L CNN
 F 1 "MC4558CN" H 8850 12450 50  0000 L CNN
-F 2 "" H 8850 12650 50  0001 C CNN
+F 2 "Package_DIP:DIP-8_W7.62mm" H 8850 12650 50  0001 C CNN
 F 3 "http://www.ti.com/lit/ds/symlink/rc4558.pdf" H 8850 12650 50  0001 C CNN
 	1    8850 12650
@@
 F 0 "U6" H 10200 10717 50  0000 C CNN
 F 1 "MC4558CN" H 10200 10626 50  0000 C CNN
-F 2 "" H 10200 10350 50  0001 C CNN
+F 2 "Package_DIP:DIP-8_W7.62mm" H 10200 10350 50  0001 C CNN
 F 3 "http://www.ti.com/lit/ds/symlink/rc4558.pdf" H 10200 10350 50  0001 C CNN
 	2    10200 10350
@@
 F 0 "U2" H 3750 16217 50  0000 C CNN
 F 1 "MC4558CN" H 3750 16126 50  0000 C CNN
-F 2 "" H 3750 15850 50  0001 C CNN
+F 2 "Package_DIP:DIP-8_W7.62mm" H 3750 15850 50  0001 C CNN
 F 3 "http://www.ti.com/lit/ds/symlink/rc4558.pdf" H 3750 15850 50  0001 C CNN
 	1    3750 15850
@@
 F 0 "U2" H 3550 18550 50  0000 L CNN
 F 1 "MC4558CN" H 3550 18150 50  0000 L CNN
-F 2 "" H 3550 18350 50  0001 C CNN
+F 2 "Package_DIP:DIP-8_W7.62mm" H 3550 18350 50  0001 C CNN
 F 3 "http://www.ti.com/lit/ds/symlink/rc4558.pdf" H 3550 18350 50  0001 C CNN
 	2    3550 18350
@@
 F 0 "U1" H 5650 6250 50  0000 L CNN
 F 1 "MC4558CN" H 5650 5850 50  0000 L CNN
-F 2 "" H 5650 6050 50  0001 C CNN
+F 2 "Package_DIP:DIP-8_W7.62mm" H 5650 6050 50  0001 C CNN
 F 3 "http://www.ti.com/lit/ds/symlink/rc4558.pdf" H 5650 6050 50  0001 C CNN
 	1    5650 6050
@@
 F 0 "U1" H 3900 7250 50  0000 L CNN
 F 1 "MC4558CN" H 3900 6850 50  0000 L CNN
-F 2 "" H 3900 7050 50  0001 C CNN
+F 2 "Package_DIP:DIP-8_W7.62mm" H 3900 7050 50  0001 C CNN
 F 3 "http://www.ti.com/lit/ds/symlink/rc4558.pdf" H 3900 7050 50  0001 C CNN
 	2    3900 7050
@@
 F 0 "U1" H 3050 5900 50  0000 L CNN
 F 1 "MC4558CN" H 3050 5500 50  0000 L CNN
-F 2 "" H 3050 5700 50  0001 C CNN
+F 2 "Package_DIP:DIP-8_W7.62mm" H 3050 5700 50  0001 C CNN
 F 3 "http://www.ti.com/lit/ds/symlink/rc4558.pdf" H 3050 5700 50  0001 C CNN
 	3    3050 5700
@@
 Non Standard 9 pin  mini DIN
 $Comp
-L SW-Texas:LM1036 U?
+L SW-Texas:LM1036 U3
 U 1 1 5E52540A
 P 9450 2400
-F 0 "U?" H 9700 2950 50  0000 C CNN
+F 0 "U3" H 9700 2950 50  0000 C CNN
 F 1 "LM1036" H 9050 2950 50  0000 C CNN
-F 2 "" H 10050 2300 50  0001 C CNN
+F 2 "Package_DIP:DIP-20_W7.62mm" H 10050 2300 50  0001 C CNN
 F 3 "" H 8650 2350 50  0001 C CNN
 	1    9450 2400
@@
 F 0 "U2" H 1500 17100 50  0000 L CNN
 F 1 "MC4558CN" H 1500 16700 50  0000 L CNN
-F 2 "" H 1500 16900 50  0001 C CNN
+F 2 "Package_DIP:DIP-8_W7.62mm" H 1500 16900 50  0001 C CNN
 F 3 "http://www.ti.com/lit/ds/symlink/rc4558.pdf" H 1500 16900 50  0001 C CNN
 	3    1500 16900
@@
 F 0 "U6" H 10800 13000 50  0000 L CNN
 F 1 "MC4558CN" H 10800 12600 50  0000 L CNN
-F 2 "" H 10800 12800 50  0001 C CNN
+F 2 "Package_DIP:DIP-8_W7.62mm" H 10800 12800 50  0001 C CNN
 F 3 "http://www.ti.com/lit/ds/symlink/rc4558.pdf" H 10800 12800 50  0001 C CNN
 	3    10800 12800
