File: 2-speaker-subwoofer/amplifier-pcb-no-jumpers/amplifier-pcb.sch (KiCad schematic (older format))
At the start: 154 parts, among them J3 CUI_PD-30, J4 RIGHT SPEAKER, J5 SUB OUT, J6 AUDIO_IN, Q3 2SA1015, Q4 2SK192A, Q5 2SC1815, Q6 2SC1815, U1 MC4558CN, U10 STA7360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

Commit message: copying modifications from original to no jumper version
Parts:
- D1, D2: value D -> 1N4148
- D3, D4, D5, D6, D7: value D -> 6A2; Characteristics (none) -> 200V Peak Reverse Voltage, 140VRMS max, 200V max DC blockin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; Description (none) -> power diode
- Q4: Manufacturer (none) -> Toshiba; Package ID (none) -> 2-4E1D Toshiba
- U1, U2, U6: footprint (none) -> Package_DIP:DIP-8_W7.62mm
- U3: renamed from U?; footprint (none) -> Package_DIP:DIP-20_W7.62mm
Connections:
- net S_GND: now reaches C37.2, J4.5 (Pin_5), JP2.2, R26.1, R37.1
- net IN1 renamed LEFT_IN
- net IN2 renamed RIGHT_IN
- net OUT1 renamed LEFT
- net OUT1_AMP renamed L_SPK
- net OUT1_PRE renamed LEFT_PRE
- net OUT2 renamed RIGHT
- net OUT2_AMP renamed R_SPK
- net OUT2_PRE renamed RIGHT_PRE
- net PIN3 renamed ZENER_VREF
- net PIN4 renamed SUB_RETURN
- net PIN6 renamed PWR_ON
Other:
- note added: "Female to Male pin # \ncross reference\n1 = 3\n2 = 2\n3 = 1\n4 = 7\n5 = 6\n6 = 5\n7 = 4\n8 = 9\n9 = 8"
- note added: "MINI DIN 9\npin numbering\nlooking into the \nfemale board \nconnector\n 1 - 2 - 3\n4 - 5 - 6 -7\n 8 - 9"
- note added: "OUT1 = L\nOUT2 = R"
- note added: "PWR_ON is signal\nfrom right speaker\nto turn power on"
- note added: "wire colors to mini din male pins\nnumbered looking into the connector\non the cable\n 1 - 2 - 3\n4 - 5 - 6 - 7\n 8 - 9\n\nblack = shield\nwhite = 3\ngrey = 2\nbrown = 8\npurple = 1\nblue = 7\ngreen = 6\nyellow = 5\norange = 4\nred = 9"
- note removed: "MINI DIN 9\npin numbering\n 1 - 2 - 3\n4 - 5 - 6 -7\n 8 - 9"
- moved on the sheet: C10, C100, C101, C105, C106, C11, C12, C13, C21, C22, C23, C24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

Commit message: banished all jumpers
swapped all GNDS to GND symbols due to jumpers being banished
Parts:
- removed JP1, JP11, JP13, JP14, JP15, JP16, JP17, JP18, JP19, JP2, JP20, JP21, JP22, JP23, JP24, JP25, JP26, JP3, JP4, JP5, JP6, JP7, JP8: Jumper, symbol Device:Jumper
Connections:
- net GNDS is gone; now on net GND: C103.2, C104.2, C39.2, C44.2, C45.2, C46.1, C47.2, R62.2, R70.1, R80.1, U6.4 (V-), U9.3 (S-GND)
- net S_GND is gone; now on net GND: C37.2, J4.5 (Pin_5), R26.1, R37.1
- net +12V: now also C36.1, D7.1 (K), Q5.2 (C), Q6.2 (C), U6.8 (V+)
- net +VDC: now also R71.1
- net Bass_Cnt: now also R1.1
- net GND: now also U10.3 (S-GND)
- net LEFT: now also C45.1, R44.2
- net PWR_ON: now also R41.2
- net RIGHT: now also C44.1, R43.2
- net STANDBY: now also C39.1, R79.1, R80.2
- net SUB-OUT-AMP: now also J5.2 (Pin_2)
- net Treble_Cnt: now also R2.2
- net Volume_Cnt: now also R3.1
- net ZENER_VREF: now also R19.2, U3.17 (Zener_Voltage), U3.7 (Loudness_Comp_Cnt)
- net at C37.1, R18.2, R34.2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: now also R48.1, R63.1, R68.1
- net at R63.2: now also C63.1, Q6.3 (B)
- net at Q3.3 (B), R38.1: now also R41.1
- net at C31.1, R30.2, U2.7: now also C49.1
- net at C13.2, R11.2, U2.1: now also C38.1
- net at C105.1, U3.13 (OUt2): now also R75.1
Other:
- note removed: "GND and GNDS are equivalent,\nUsing different symbols due to the jumpers"
- moved on the sheet: R41
