File: acoustic-research-advent-powered-partner-570/power-input-board.sch (KiCad schematic (older format))
At the start: 0 parts

Commit message: Amp board should be complete, working on input board
Parts:
- added C1: 1nF, symbol Device:C_Small
- added C19: 47nF 20%, symbol Device:C_Small
- added D14: A465401, symbol Device:D
- added J24: DNP, symbol Device:Jumper_NC_Small
- added J?: JUMPER_TO_AMP_BOARD, symbol Connector_Generic:Conn_01x06
- added J?: Conn_WallSocket, symbol Connector:Conn_WallSocket
- added J?: Barrel_Jack, symbol Connector:Barrel_Jack
- added J?: Signal Input, symbol Connector:Conn_Coaxial
- added P?: Conn_WallPlug, symbol Connector:Conn_WallPlug
- added R23: 2k2Ω 5% 0.25W, symbol Device:R_Small_US
- added SK1: AC Out, symbol Connector_Generic:Conn_01x04
- added SW?: MAIN POWER, symbol Switch:SW_DPST
Connections:
- new net: SK1.1 (Pin_1), SK1.4 (Pin_4)
- new net: SK1.2 (Pin_2), SW?.2
- new net: C1.1, J?.1 (Pin_1), R23.1
- new net: J?.1 (In), R23.2
- new net: C1.2, C19.2, J?.2 (Ext), J?.2 (Pin_2)
- new net: D14.1 (K), J?.5 (Pin_5), J?.6 (Pin_6)
- new net: D14.2 (A), SW?.3
- new net: J?.1 (AC_P), P?.1 (AC_P), SW?.1
- new net: J?.2 (AC_N), P?.2 (AC_N)
- new net Earth_Protective: C19.1, J24.1, J24.2
- no-connect marks 0 -> 1
Other:
- note added: "115V 230V"
- note added: "All One Connector"
- note added: "PIN 6 is White Stripe"
