File: acoustic-research-advent-powered-partner-570/amp-board.sch (KiCad schematic (older format))
At the start: 145 parts, among them Q1 C546B, Q10 C546B, Q11 C546B, Q12 C556B, Q13 BC33740, Q14 C556B, Q15 KSE3055T, Q16 KSE3055T, Q17 KSE3055T, Q18 BC33740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

Commit message: more transistor connections
Parts:
- added C10: 10uF 35V +85C vent, symbol Device:CP1_Small
- added D13: 1N4148, symbol Device:D_Small
- added R10: 470kΩ 5% 0.25W, symbol Device:R_Small_US
- added R11: 150Ω 5% 0.25W, symbol Device:R_Small_US
- added R12: 33kΩ 5% 0.25W, symbol Device:R_Small_US
- added R18: 2k2Ω 5% 0.25W, symbol Device:R_Small_US
Connections:
- net at Q7.1 (C): now also R15.1
- net at Q7.2 (B): now also D7.1 (K), R14.1, C10.2
- net at Q8.3 (E): now also Q9.2 (B)
- net at Q10.1 (C): now also Q11.2 (B), R22.2
- net at Q10.2 (B): now also D13.2 (A)
- net at C16.2, C21.2, C27.2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: now also R13.2; no longer R13.1
- net at D6.1 (K): now also R18.1
- net at R19.2: now also J?.1 (Pin_1), R18.2
- net at U1.1: now also R10.1, R12.1
- net at U1.2 (-): now also R10.2, R11.1
- net at C9.1: now also R11.2
- net at R21.2: now also C12.1, D13.1 (K)
- new net: C10.1, R12.2, R13.1
Other:
- moved on the sheet: BK, BL, C12, C17, C18, C23, C24, C25, C28, C31, C9, D10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

Commit message: Amp board should be complete, working on input board
Parts:
- added H?: Bracket Screw, symbol Mechanical:MountingHole_Pad
- added H?: Other Bracket Screw, symbol Mechanical:MountingHole_Pad
- added R60: 1k2Ω 2% 0.25W, symbol Device:R_Small_US
- added R66: 680Ω 5% 0.25W, symbol Device:R_Small_US
- U1: value NJM4558 -> 4558DD
- U2: value NJM4556A -> 4556D
Connections:
- net at C29.1, J16.2, J?.5 (Pin_5)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: now also R65.1; no longer R65.2
- net at Q1.2 (B): now also C16.1, R65.2
- net at Q8.2 (B), R16.1: no longer R20.2
- net at C23.1, J10.2, U2.2 (-): now also C28.2
- net at U2.6 (-): now also R46.2, R60.1
- net at C16.2, C21.2, C27.2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: now also R66.2
- net at C28.1: now also R66.1
- net at C21.1: now also R60.2
- net at C12.1, D13.1 (K), R21.2: now also R20.2
- no-connect marks 1 -> 3
Other:
- moved on the sheet: C16, C21, C23, C28, R13, R20, R65

Commit message: adding some footprints
Parts:
- BK, BL, JP? (x2), RD, YL: footprint (none) -> Connector_PinHeader_2.54mm:PinHeader_1x01_P2.54mm_Vertical
- Q15, Q16, Q17, Q3: footprint TO-220-3 -> Package_TO_SOT_THT:TO-220-3_Vertical
- U1, U2: footprint (none) -> Package_DIP:DIP-8_W7.62mm
Changed lines of the file:
@@
 F 0 "Q16" H 12541 14296 50  0000 L CNN
 F 1 "KSE3055T" H 12541 14205 50  0000 L CNN
-F 2 "TO-220-3" H 12550 14350 50  0001 C CNN
+F 2 "Package_TO_SOT_THT:TO-220-3_Vertical" H 12550 14350 50  0001 C CNN
 F 3 "~" H 12350 14250 50  0001 C CNN
 	1    12350 14250
@@
 F 0 "Q17" H 12541 15596 50  0000 L CNN
 F 1 "KSE3055T" H 12541 15505 50  0000 L CNN
-F 2 "TO-220-3" H 12550 15650 50  0001 C CNN
+F 2 "Package_TO_SOT_THT:TO-220-3_Vertical" H 12550 15650 50  0001 C CNN
 F 3 "~" H 12350 15550 50  0001 C CNN
 	1    12350 15550
@@
 F 0 "Q15" H 7841 15146 50  0000 L CNN
 F 1 "KSE3055T" H 7841 15055 50  0000 L CNN
-F 2 "TO-220-3" H 7850 15200 50  0001 C CNN
+F 2 "Package_TO_SOT_THT:TO-220-3_Vertical" H 7850 15200 50  0001 C CNN
 F 3 "~" H 7650 15100 50  0001 C CNN
 	1    7650 15100
@@
 F 0 "Q3" H 11741 17046 50  0000 L CNN
 F 1 "KSE3055T" H 11741 16955 50  0000 L CNN
-F 2 "TO-220-3" H 11750 17100 50  0001 C CNN
+F 2 "Package_TO_SOT_THT:TO-220-3_Vertical" H 11750 17100 50  0001 C CNN
 F 3 "~" H 11550 17000 50  0001 C CNN
 	1    11550 17000
@@
 F 0 "U2" H 18450 7433 50  0000 C CNN
 F 1 "4556D" H 18450 7524 50  0000 C CNN
-F 2 "" H 18450 7800 50  0001 C CNN
+F 2 "Package_DIP:DIP-8_W7.62mm" H 18450 7800 50  0001 C CNN
 F 3 "http://www.njr.com/semicon/PDF/NJM4556A_E.pdf" H 18450 7800 50  0001 C CNN
 	1    18450 7800
@@
 F 0 "U2" H 7800 7767 50  0000 C CNN
 F 1 "4556D" H 7800 7676 50  0000 C CNN
-F 2 "" H 7800 7400 50  0001 C CNN
+F 2 "Package_DIP:DIP-8_W7.62mm" H 7800 7400 50  0001 C CNN
 F 3 "http://www.njr.com/semicon/PDF/NJM4556A_E.pdf" H 7800 7400 50  0001 C CNN
 	2    7800 7400
@@
 F 0 "U2" H 18358 6196 50  0000 L CNN
 F 1 "4556D" H 18358 6105 50  0000 L CNN
-F 2 "" H 18400 6150 50  0001 C CNN
+F 2 "Package_DIP:DIP-8_W7.62mm" H 18400 6150 50  0001 C CNN
 F 3 "http://www.njr.com/semicon/PDF/NJM4556A_E.pdf" H 18400 6150 50  0001 C CNN
 	3    18400 6150
@@
 F 0 "BK" H 18380 15142 50  0000 L CNN
 F 1 "B-" H 18380 15051 50  0000 L CNN
-F 2 "" H 18300 15100 50  0001 C CNN
+F 2 "Connector_PinHeader_2.54mm:PinHeader_1x01_P2.54mm_Vertical" H 18300 15100 50  0001 C CNN
 F 3 "~" H 18300 15100 50  0001 C CNN
 	1    18300 15100
@@
 F 0 "BL" H 18380 15392 50  0000 L CNN
 F 1 "T-" H 18380 15301 50  0000 L CNN
-F 2 "" H 18300 15350 50  0001 C CNN
+F 2 "Connector_PinHeader_2.54mm:PinHeader_1x01_P2.54mm_Vertical" H 18300 15350 50  0001 C CNN
 F 3 "~" H 18300 15350 50  0001 C CNN
 	1    18300 15350
@@
 F 0 "U1" H 12100 6317 50  0000 C CNN
 F 1 "4558DD" H 12100 6226 50  0000 C CNN
-F 2 "" H 12100 5950 50  0001 C CNN
+F 2 "Package_DIP:DIP-8_W7.62mm" H 12100 5950 50  0001 C CNN
 F 3 "http://www.njr.com/semicon/PDF/NJM4558_NJM4559_E.pdf" H 12100 5950 50  0001 C CNN
 	1    12100 5950
@@
 F 0 "U1" H 7850 2767 50  0000 C CNN
 F 1 "4558DD" H 7850 2676 50  0000 C CNN
-F 2 "" H 7850 2400 50  0001 C CNN
+F 2 "Package_DIP:DIP-8_W7.62mm" H 7850 2400 50  0001 C CNN
 F 3 "http://www.njr.com/semicon/PDF/NJM4558_NJM4559_E.pdf" H 7850 2400 50  0001 C CNN
 	2    7850 2400
@@
 F 0 "U1" H 17558 6096 50  0000 L CNN
 F 1 "4558DD" H 17558 6005 50  0000 L CNN
-F 2 "" H 17600 6050 50  0001 C CNN
+F 2 "Package_DIP:DIP-8_W7.62mm" H 17600 6050 50  0001 C CNN
 F 3 "http://www.njr.com/semicon/PDF/NJM4558_NJM4559_E.pdf" H 17600 6050 50  0001 C CNN
 	3    17600 6050
@@
 F 0 "JP?" H 9418 7425 50  0000 C CNN
 F 1 "A<" H 9418 7516 50  0000 C CNN
-F 2 "" H 9500 7650 50  0001 C CNN
+F 2 "Connector_PinHeader_2.54mm:PinHeader_1x01_P2.54mm_Vertical" H 9500 7650 50  0001 C CNN
 F 3 "~" H 9500 7650 50  0001 C CNN
 	1    9500 7650
@@
 F 0 "JP?" H 6418 8475 50  0000 C CNN
 F 1 "A<" H 6418 8566 50  0000 C CNN
-F 2 "" H 6500 8700 50  0001 C CNN
+F 2 "Connector_PinHeader_2.54mm:PinHeader_1x01_P2.54mm_Vertical" H 6500 8700 50  0001 C CNN
 F 3 "~" H 6500 8700 50  0001 C CNN
 	1    6500 8700
@@
 F 0 "RD" H 11980 17592 50  0000 L CNN
 F 1 "B+" H 11980 17501 50  0000 L CNN
-F 2 "" H 11900 17550 50  0001 C CNN
+F 2 "Connector_PinHeader_2.54mm:PinHeader_1x01_P2.54mm_Vertical" H 11900 17550 50  0001 C CNN
 F 3 "~" H 11900 17550 50  0001 C CNN
 	1    11900 17550
@@
 F 0 "YL" H 11930 18142 50  0000 L CNN
 F 1 "T+" H 11930 18051 50  0000 L CNN
-F 2 "" H 11850 18100 50  0001 C CNN
+F 2 "Connector_PinHeader_2.54mm:PinHeader_1x01_P2.54mm_Vertical" H 11850 18100 50  0001 C CNN
 F 3 "~" H 11850 18100 50  0001 C CNN
 	1    11850 18100

Commit message: trying to clean schematic up a bit
Connections:
- net +VDC: now reaches C29.1, J16.2, J?.5 (Pin_5), J?.6 (Pin_6), Q1.1 (C), R65.1
- net AUDIO_GND: now reaches C12.2, J8.1, J?.2 (Pin_2), Q10.3 (E), Q11.3 (E), R21.1, R25.1
- net at J15.1, R51.2: now also J17.2; no longer J17.1
- net AUDIO_IN: now reaches J?.1 (Pin_1), R24.2, R49.2
- net GND: now reaches C29.2, J?.3 (Pin_3), J?.4 (Pin_4)
- net GND: now also J17.1; no longer J17.2
Other:
- moved on the sheet: C29, J17, J?
Changed lines of the file:
@@
 	17550 8950 17550 8850
 Wire Wire Line
-	17550 8850 12950 8850
-Wire Wire Line
-	12950 8850 12950 6550
-Wire Wire Line
-	12950 6550 18700 6550
+	17550 8850 15700 8850
+Wire Wire Line
+	15700 8850 15700 6550
+Wire Wire Line
+	15700 6550 18700 6550
 Wire Wire Line
 	18700 6550 18700 6450
@@
 L Connector_Generic:Conn_01x06 J?
 U 1 1 5F37CABD
-P 5950 5000
-F 0 "J?" H 6030 4992 50  0000 L CNN
-F 1 "JUMPER_TO_INPUT_BOARD" H 6030 4901 50  0000 L CNN
-F 2 "" H 5950 5000 50  0001 C CNN
-F 3 "~" H 5950 5000 50  0001 C CNN
-	1    5950 5000
+P 2950 5000
+F 0 "J?" H 3030 4992 50  0000 L CNN
+F 1 "JUMPER_TO_INPUT_BOARD" H 3030 4901 50  0000 L CNN
+F 2 "" H 2950 5000 50  0001 C CNN
+F 3 "~" H 2950 5000 50  0001 C CNN
+	1    2950 5000
 	-1   0    0    -1
 $EndComp
-Text Notes 5850 4900 2    50   ~ 0
+Text Notes 2850 4900 2    50   ~ 0
 PIN 6 is White Stripe
 Wire Wire Line
 	6850 4900 6850 4250
 Wire Wire Line
-	6150 4900 6850 4900
+	3150 4900 6850 4900
 Connection ~ 6850 4250
 Wire Wire Line
@@
 L Device:CP1_Small C29
 U 1 1 5F3D458D
-P 6700 5550
-F 0 "C29" V 6472 5550 50  0000 C CNN
-F 1 "1uF 35V +85C vent" V 6563 5550 50  0000 C CNN
-F 2 "" H 6700 5550 50  0001 C CNN
-F 3 "~" H 6700 5550 50  0001 C CNN
-	1    6700 5550
-	0    1    1    0
-$EndComp
-Wire Wire Line
-	6150 5000 6300 5000
-Wire Wire Line
-	6300 5000 6300 5100
-Wire Wire Line
-	6300 5100 6150 5100
-Wire Wire Line
-	6600 5550 6500 5550
-Wire Wire Line
-	6500 5550 6500 5100
-Wire Wire Line
-	6500 5100 6300 5100
-Connection ~ 6300 5100
+P 4150 5200
+F 0 "C29" V 3922 5200 50  0000 C CNN
+F 1 "1uF 35V +85C vent" V 4013 5200 50  0000 C CNN
+F 2 "" H 4150 5200 50  0001 C CNN
+F 3 "~" H 4150 5200 50  0001 C CNN
+	1    4150 5200
+	-1   0    0    1
+$EndComp
+Wire Wire Line
+	3150 5000 3250 5000
+Wire Wire Line
+	3250 5000 3250 5100
+Wire Wire Line
+	3250 5100 3150 5100
+Wire Wire Line
+	5450 5100 5400 5100
+Connection ~ 3250 5100
 $Comp
 L Device:Jumper_NC_Small J17
 U 1 1 5F40EBDD
-P 6300 5650
-F 0 "J17" H 6300 5771 50  0000 C CNN
-F 1 "~" H 6300 5771 50  0000 C CNN
-F 2 "" H 6300 5650 50  0001 C CNN
-F 3 "~" H 6300 5650 50  0001 C CNN
-	1    6300 5650
-	1    0    0    -1
-$EndComp
-Wire Wire Line
-	6400 5650 6500 5650
-Wire Wire Line
-	6500 5650 6500 5550
-Connection ~ 6500 5550
+P 5300 5100
+F 0 "J17" H 5300 5221 50  0000 C CNN
+F 1 "~" H 5300 5221 50  0000 C CNN
+F 2 "" H 5300 5100 50  0001 C CNN
+F 3 "~" H 5300 5100 50  0001 C CNN
+	1    5300 5100
+	1    0    0    -1
+$EndComp
 Wire Wire Line
 	10150 12700 10150 12900
@@
 $EndComp
 Wire Wire Line
-	5450 5650 5450 14650
-Wire Wire Line
 	5450 14650 6500 14650
 Wire Wire Line
@@
 	11200 9550 11500 9550
 Wire Wire Line
-	6800 5550 6900 5550
-Wire Wire Line
-	6900 5550 6900 8000
-Wire Wire Line
 	6900 8000 9600 8000
 Wire Wire Line
@@
 	11900 8200 11900 9550
 Wire Wire Line
-	6900 5550 6900 5300
-Wire Wire Line
-	6900 5300 6300 5300
-Connection ~ 6900 5550
-Wire Wire Line
-	6150 5200 6300 5200
-Wire Wire Line
-	6300 5200 6300 5300
-Connection ~ 6300 5300
-Wire Wire Line
-	6300 5300 6150 5300
+	6900 5300 5850 5300
+Wire Wire Line
+	3150 5200 3250 5200
+Wire Wire Line
+	3250 5200 3250 5300
+Connection ~ 3250 5300
+Wire Wire Line
+	3250 5300 3150 5300
 Wire Wire Line
 	11450 8200 11450 6600
@@
 Connection ~ 6400 4800
 Wire Wire Line
-	6400 4800 6150 4800
+	6400 4800 3150 4800
 Wire Wire Line
 	6600 4600 7850 4600
@@
 	8000 3950 8100 3950
 Wire Wire Line
-	8100 3950 8100 3200
-Wire Wire Line
-	8100 3200 7250 3200
-Wire Wire Line
 	6500 3200 6500 3700
 $Comp
@@
 	1    0    0    -1
 $EndComp
-Wire Wire Line
-	7250 3050 7250 3200
-Connection ~ 7250 3200
-Wire Wire Line
-	7250 3200 6500 3200
 Wire Wire Line
 	7250 2850 7250 2750
@@
 	5950 6450 5950 6650
 Wire Wire Line
-	5450 5650 6200 5650
-Wire Wire Line
 	7250 5750 5950 5750
 Wire Wire Line
@@
 	6150 8300 5950 8300
 Wire Wire Line
-	5500 8700 5500 8450
-Wire Wire Line
-	5500 8450 5600 8450
+	5600 8700 5600 8450
 Wire Wire Line
 	9900 6400 9900 7650
@@
 	5600 8450 5650 8450
 Wire Wire Line
-	5500 8700 5850 8700
+	5600 8700 5850 8700
 $Comp
 L Device:R_Small_US R19
@@
 NoConn ~ 10650 10900
 NoConn ~ 11000 10900
+Text Label 3250 4800 0    50   ~ 0
+AUDIO_IN
+Text Label 3250 4900 0    50   ~ 0
+AUDIO_GND
+Wire Wire Line
+	7250 3200 6500 3200
+Wire Wire Line
+	7250 3050 7250 3200
+Connection ~ 7250 3200
+Wire Wire Line
+	8100 3950 8100 3200
+Wire Wire Line
+	8100 3200 7250 3200
+$Comp
+L power:GND #PWR?
+U 1 1 65AFA5F3
+P 3800 5200
+F 0 "#PWR?" H 3800 4950 50  0001 C CNN
+F 1 "GND" H 3805 5027 50  0000 C CNN
+F 2 "" H 3800 5200 50  0001 C CNN
+F 3 "" H 3800 5200 50  0001 C CNN
+	1    3800 5200
+	1    0    0    -1
+$EndComp
+Wire Wire Line
+	3800 5200 3800 5100
+Connection ~ 3800 5100
+Wire Wire Line
+	3800 5100 3250 5100
+Connection ~ 4150 5300
+Wire Wire Line
+	4150 5300 3250 5300
+Connection ~ 4150 5100
+Wire Wire Line
+	4150 5100 3800 5100
+Wire Wire Line
+	6900 5300 6900 8000
+Wire Wire Line
+	5200 5100 4150 5100
+Wire Wire Line
+	5450 5100 5450 14650
+$Comp
+L power:+VDC #PWR?
+U 1 1 65D58178
+P 5850 5250
+F 0 "#PWR?" H 5850 5150 50  0001 C CNN
+F 1 "+VDC" H 5850 5525 50  0000 C CNN
+F 2 "" H 5850 5250 50  0001 C CNN
+F 3 "" H 5850 5250 50  0001 C CNN
+	1    5850 5250
+	1    0    0    -1
+$EndComp
+Wire Wire Line
+	5850 5250 5850 5300
+Connection ~ 5850 5300
+Wire Wire Line
+	5850 5300 4150 5300
 $EndSCHEMATC
