File: acoustic-research-advent-powered-partner-570/acoustic-research-advent-powered-partner-570/amp-board.sch (KiCad schematic (older format))
At the start: 155 parts, among them Q1 C546B, Q10 C546B, Q11 C546B, Q12 C556B, Q13 BC33740, Q14 C556B, Q15 KSE3055T, Q16 KSE3055T, Q17 KSE3055T, Q18 BC33740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

Commit message: moved original schematics into their own folder, also fixed R17 connections
Connections:
- net at Q8.2 (B), R16.1: now also R17.2
Changed lines of the file:
@@
 Connection ~ 6750 3350
 Wire Wire Line
-	12050 7600 12350 7600
+	12050 7600 12250 7600
 Wire Wire Line
 	14550 7050 14550 7150
@@
 Wire Wire Line
 	5850 5300 4150 5300
+Wire Wire Line
+	10350 7150 10250 7150
+Wire Wire Line
+	10250 7150 10250 7300
+Wire Wire Line
+	10250 7300 12250 7300
+Wire Wire Line
+	12250 7300 12250 7600
+Connection ~ 12250 7600
+Wire Wire Line
+	12250 7600 12350 7600
 $EndSCHEMATC
