File: acoustic-research-advent-powered-partner-570/acoustic-research-advent-powered-partner-570-no-jumpers/amp-board.sch (KiCad schematic (older format))
At the start: 151 parts, among them Q1 C546B, Q10 C546B, Q11 C546B, Q12 C556B, Q13 BC33740, Q14 C556B, Q15 KSE3055T, Q16 KSE3055T, Q17 KSE3055T, Q18 BC33740, Q2 BC32740, Q3 KSE3055T, Q4 C546B, Q5 BC32740, Q6 C546B, Q7 C546B, Q8 C546B, Q9 C546B, U1 4558DD, U2 4556D

Commit message: simplified speghetti by using power rail symbols
Parts:
- removed J1, J10, J11, J12, J13, J14, J16, J18, J20, J21, J22, J8, J9: ~, symbol Device:Jumper_NC_Small
Connections:
- net +VDC is gone; now on net VBUS: C29.1, J?.5 (Pin_5), J?.6 (Pin_6), Q1.1 (C), R65.1
- net AUDIO_GND is gone; now on net GND: C12.2, J?.2 (Pin_2), Q10.3 (E), Q11.3 (E), R21.1, R25.1
- net GND: now also C16.2, C2.2, C21.2, C24.2, C25.2, C27.2, C6.1, C7.1, C9.2, D1.2 (-), D7.2 (A), H?.1, J?.2 (Pin_2), Q7.3 (E), R13.2, R14.2, R35.2, R41.2, R47.2, R55.1, R63.1, R66.2, R68.1, U1.4 (V-), U2.4 (V-)
- net NEUT: now reaches C3.2, D1.4 (~~), SK2.2 (Pin_2)
- net LINE: now reaches C3.1, FUSE.2
- net LINE: now also D1.3 (~~)
- net VBUS: now reaches C2.1, D1.1 (+), R6.2
- net VBUS: now also R3.1, R53.2, R54.2
- net at Q1.3 (E), R48.1: now also C11.1, Q9.3 (E), R17.1, R19.1, R22.1, U1.8 (V+), U2.8 (V+)
- net at R61.1: now also C23.1, C28.2, U2.2 (-)
- net at C26.2, C27.1, R26.1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: now also R7.1
Other:
- moved on the sheet: R56, R?

Commit message: a little bit more cleanup
Other:
- moved on the sheet: R44, R55
Changed lines of the file:
@@
 L Device:R_Small_US R55
 U 1 1 5E8DFA91
-P 9800 12900
-F 0 "R55" V 9595 12900 50  0000 C CNN
-F 1 "0.22Ω 5% 1W" V 9686 12900 50  0000 C CNN
-F 2 "" H 9800 12900 50  0001 C CNN
-F 3 "~" H 9800 12900 50  0001 C CNN
-	1    9800 12900
-	0    1    1    0
+P 12300 15950
+F 0 "R55" V 12095 15950 50  0000 C CNN
+F 1 "0.22Ω 5% 1W" V 12186 15950 50  0000 C CNN
+F 2 "" H 12300 15950 50  0001 C CNN
+F 3 "~" H 12300 15950 50  0001 C CNN
+	1    12300 15950
+	-1   0    0    1
 $EndComp
 $Comp
@@
 L Device:R_Small_US R44
 U 1 1 5E946126
-P 13050 13550
-F 0 "R44" V 12845 13550 50  0000 C CNN
-F 1 "100Ω 5% 0.25W" V 12936 13550 50  0000 C CNN
-F 2 "" H 13050 13550 50  0001 C CNN
-F 3 "~" H 13050 13550 50  0001 C CNN
-	1    13050 13550
+P 19050 13550
+F 0 "R44" V 18845 13550 50  0000 C CNN
+F 1 "100Ω 5% 0.25W" V 18936 13550 50  0000 C CNN
+F 2 "" H 19050 13550 50  0001 C CNN
+F 3 "~" H 19050 13550 50  0001 C CNN
+	1    19050 13550
 	-1   0    0    1
 $EndComp
 Wire Wire Line
-	13050 13450 13050 13200
-Wire Wire Line
-	13050 13200 17250 13200
-Wire Wire Line
 	17250 13200 17250 13150
 Wire Wire Line
@@
 Wire Wire Line
 	19050 13200 17250 13200
-Connection ~ 17250 13200
 $Comp
 L Device:R_Small_US R50
@@
 	19950 9700 19950 13850
 Wire Wire Line
-	19950 13850 18450 13850
-Wire Wire Line
-	13050 13850 13050 13650
+	19950 13850 19050 13850
 Wire Wire Line
 	18450 12900 18450 13850
-Connection ~ 18450 13850
-Wire Wire Line
-	18450 13850 13050 13850
 $Comp
 L Amplifier_Operational:NJM4556A U2
@@
 Connection ~ 3250 5100
 Wire Wire Line
-	10150 12900 9900 12900
-Wire Wire Line
-	9700 16200 12300 16200
-Wire Wire Line
-	12300 16200 12300 15750
+	12300 16200 12300 16050
 Connection ~ 12300 15750
 Wire Wire Line
@@
 	7200 13950 7500 13950
 Wire Wire Line
-	9700 12900 9700 16200
-Wire Wire Line
 	8700 14000 10000 14000
 Wire Wire Line
@@
 L power:GND #PWR?
 U 1 1 60874B09
-P 10150 13000
-F 0 "#PWR?" H 10150 12750 50  0001 C CNN
-F 1 "GND" H 10155 12827 50  0000 C CNN
-F 2 "" H 10150 13000 50  0001 C CNN
-F 3 "" H 10150 13000 50  0001 C CNN
-	1    10150 13000
-	1    0    0    -1
-$EndComp
-Wire Wire Line
-	10150 13000 10150 12900
+P 12300 16200
+F 0 "#PWR?" H 12300 15950 50  0001 C CNN
+F 1 "GND" H 12305 16027 50  0000 C CNN
+F 2 "" H 12300 16200 50  0001 C CNN
+F 3 "" H 12300 16200 50  0001 C CNN
+	1    12300 16200
+	1    0    0    -1
+$EndComp
 $Comp
 L power:GND #PWR?
@@
 	9600 9200 9600 9150
 Connection ~ 9600 9150
+Wire Wire Line
+	12300 15850 12300 15750
+Wire Wire Line
+	19050 13450 19050 13200
+Connection ~ 19050 13200
+Wire Wire Line
+	19050 13650 19050 13850
+Connection ~ 19050 13850
+Wire Wire Line
+	19050 13850 18450 13850
 $EndSCHEMATC

Commit message: more simplificatoin
Other:
- moved on the sheet: Q13, Q9, R52

Commit message: added some text notes on schematic
Other:
- note added: "Darlington Pair"
- note added: "Darlington Pair\nwith bypass bleedoff\nresistor"
Changed lines of the file:
@@
 Wire Wire Line
 	7000 14700 7100 14700
+Text Notes 8250 14850 0    50   ~ 0
+Darlington Pair\nwith bypass bleedoff\nresistor
+Text Notes 12700 7250 0    50   ~ 0
+Darlington Pair
 $EndSCHEMATC

Commit message: changes
Connections:
- net AUDIO_IN: now also R24.1; no longer R24.2
- net GND: now also R13.1; no longer R13.2
- net at R51.1: now also C18.2; no longer C18.1
- net at C10.1, R12.2: now also R13.2; no longer R13.1
- net at R25.3: now also R24.2; no longer R24.1
- net at C17.2: now also C18.1; no longer C18.2
Other:
- note added: "complimentary feedback pair - \nPNP with bypass resistor"
- moved on the sheet: C17, C18, C9, Q16, Q17, Q2, Q5, R10, R11, R12, R13, R24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
