File: gamestop-av-switch/gamestop-av-switch.sch (KiCad schematic (older format))
At the start: 0 parts

Commit message: Starting to wire up switches
Using 01x09 connectors until I figure out what the internal switch
wiring is

Added Jumper library
Parts:
- added J1, J13, J17, J19, J30, J33, J34, J35, J36, J38, J40, J41, J42, J45, J46, J7: ~, symbol Jumper:Jumper_2_Bridged
- added J?: SW1_L, symbol Connector_Generic:Conn_01x09
- added J?: SW1_R, symbol Connector_Generic:Conn_01x09
- added J?: SW2_L, symbol Connector_Generic:Conn_01x09
- added J?: SW2_R, symbol Connector_Generic:Conn_01x09
- added J?: SW3_L, symbol Connector_Generic:Conn_01x09
- added J?: SW3_R, symbol Connector_Generic:Conn_01x09
- added J?: SW4_L, symbol Connector_Generic:Conn_01x09
- added J?: SW4_R, symbol Connector_Generic:Conn_01x09
- added J?: SW5_L, symbol Connector_Generic:Conn_01x09
- added J?: SW5_R, symbol Connector_Generic:Conn_01x09
- added J?: SW6_L, symbol Connector_Generic:Conn_01x09
- added J?: SW6_R, symbol Connector_Generic:Conn_01x09
- added J?: SW7_L, symbol Connector_Generic:Conn_01x09
- added J?: SW7_R, symbol Connector_Generic:Conn_01x09
Connections:
- net Front Input/C: now also J?.3 (Pin_3)
- net Front Input/Composite: now also J?.9 (Pin_9)
- net Front Input/Left: now also J?.3 (Pin_3)
- net Front Input/Right: now also J?.9 (Pin_9)
- net Front Input/Y: now also J?.6 (Pin_6)
- net Output/C: now also J35.2 (B), J40.2 (B), J45.2 (B), J?.2 (Pin_2)
- net Output/Composite: now also J1.1 (A)
- net Output/Left: now also J19.2 (B), J38.2 (B), J42.2 (B), J?.2 (Pin_2)
- net Output/Right: now also J?.8 (Pin_8), J?.8 (Pin_8), J?.8 (Pin_8), J?.8 (Pin_8)
- net Output/Y: now also J36.2 (B), J41.2 (B), J46.2 (B), J?.5 (Pin_5)
- new net: J40.1 (A), J?.2 (Pin_2)
- new net: J38.1 (A), J?.5 (Pin_5)
- new net: J41.1 (A), J?.2 (Pin_2)
- new net: J34.1 (A), J?.5 (Pin_5)
- new net: J45.1 (A), J?.2 (Pin_2)
- new net: J42.1 (A), J?.5 (Pin_5)
- new net: J46.1 (A), J?.2 (Pin_2)
- new net: J30.1 (A), J?.5 (Pin_5)
- new net: J35.1 (A), J?.2 (Pin_2)
- new net: J19.1 (A), J?.5 (Pin_5)
- new net: J36.1 (A), J?.2 (Pin_2)
- new net: J17.2 (B), J?.5 (Pin_5)
- new net: J?.4 (Pin_4), J?.5 (Pin_5), J?.6 (Pin_6)
- new net: J33.1 (A), J?.8 (Pin_8)
- new net: J13.2 (B), J17.1 (A), J33.2 (B)
- new net: J13.1 (A), J30.2 (B), J7.2 (B)
- new net: J1.2 (B), J34.2 (B), J7.1 (A)
- no-connect marks 0 -> 5
Other:
- note added: "Switches are numbered 1-7 from left to right\nlooking at the top of the PCB\n\nPins are numbered top to bottom looking at\nbottom of PCB with connectors towards the front"

Commit message: Finished Switch 6 wiring
Also added no-connects to all switches
Parts:
- added J10, J14, J15, J16, J2, J24, J25, J28, J29, J3, J4, J8, J9: ~, symbol Jumper:Jumper_2_Bridged
Connections:
- net Input 3/Blue: now also J?.9 (Pin_9)
- net Input 3/Composite: now also J?.6 (Pin_6)
- net Input 3/Green: now also J?.3 (Pin_3)
- net Input 3/Red: now also J?.6 (Pin_6)
- net Input 3/Right: now also J?.9 (Pin_9)
- net Input 3/Y: now also J?.3 (Pin_3)
- net Output/Blue: now also J2.2 (B)
- net Output/Green: now also J4.2 (B)
- net Output/Red: now also J3.2 (B)
- net at J?.2 (Pin_2): now also J10.2 (B), J4.1 (A)
- net at J?.5 (Pin_5): now also J25.1 (A)
- net at J?.8 (Pin_8): now also J24.1 (A)
- net at J?.2 (Pin_2): now also J10.1 (A), J14.2 (B)
- net at J?.5 (Pin_5): now also J28.1 (A)
- net at J?.8 (Pin_8): now also J29.1 (A)
- net at J?.2 (Pin_2): now also J14.1 (A)
- net at J?.5 (Pin_5): now also J15.1 (A)
- net at J?.8 (Pin_8): now also J16.1 (A)
- new net: J16.2 (B), J29.2 (B), J8.1 (A)
- new net: J2.1 (A), J24.2 (B), J8.2 (B)
- new net: J15.2 (B), J28.2 (B), J9.1 (A)
- new net: J25.2 (B), J3.1 (A), J9.2 (B)
- no-connect marks 5 -> 41

Commit message: Finished wiring switch 5
Parts:
- added J11, J12, J18, J20, J21, J22, J23, J26, J27, J31, J32, J37, J39, J43, J44, J47, J5, J6: ~, symbol Jumper:Jumper_2_Bridged
Connections:
- net Input 3/1: now also J?.9 (Pin_9)
- net Input 3/2: now also J?.9 (Pin_9)
- net Input 3/3: now also J?.6 (Pin_6)
- net Input 3/6: now also J?.3 (Pin_3)
- net Input 3/C: now also J?.3 (Pin_3)
- net Input 3/Left: now also J?.6 (Pin_6)
- net Output/1: now also J21.2 (B)
- net Output/2: now also J20.1 (A)
- net Output/3: now also J18.1 (A), J39.2 (B), J44.2 (B)
- net Output/6: now also J37.2 (B), J43.2 (B), J47.1 (A)
- net at J?.2 (Pin_2): now also J37.1 (A)
- net at J?.5 (Pin_5): now also J39.1 (A)
- net at J?.8 (Pin_8): now also J22.1 (A)
- net at J?.8 (Pin_8): now also J23.1 (A)
- net at J?.2 (Pin_2): now also J43.1 (A)
- net at J?.5 (Pin_5): now also J44.1 (A)
- net at J?.8 (Pin_8): now also J26.1 (A)
- net at J?.8 (Pin_8): now also J27.1 (A)
- net at J?.2 (Pin_2): now also J47.2 (B)
- net at J?.5 (Pin_5): now also J18.2 (B)
- net at J?.8 (Pin_8): now also J32.2 (B)
- net at J?.8 (Pin_8): now also J31.1 (A)
- new net: J12.1 (A), J31.2 (B)
- new net: J12.2 (B), J27.2 (B), J6.1 (A)
- new net: J21.1 (A), J23.2 (B), J6.2 (B)
- new net: J11.2 (B), J32.1 (A)
- new net: J11.1 (A), J26.2 (B), J5.2 (B)
- new net: J20.2 (B), J22.2 (B), J5.1 (A)
Other:
- moved on the sheet: J1, J10, J13, J14, J15, J16, J17, J19, J2, J24, J25, J28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

Commit message: Finished wiring switch 4
Connections:
- net Input 2/Blue: now also J?.9 (Pin_9)
- net Input 2/Composite: now also J?.6 (Pin_6)
- net Input 2/Green: now also J?.3 (Pin_3)
- net Input 2/Red: now also J?.6 (Pin_6)
- net Input 2/Right: now also J?.9 (Pin_9)
- net Input 2/Y: now also J?.3 (Pin_3)
Other:
- moved on the sheet: J11, J12, J18, J20, J22, J23, J26, J27, J31, J32, J39, J44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

Commit message: Finished wiring switch 3
Connections:
- net Input 2/1: now also J?.9 (Pin_9)
- net Input 2/2: now also J?.9 (Pin_9)
- net Input 2/3: now also J?.6 (Pin_6)
- net Input 2/6: now also J?.3 (Pin_3)
- net Input 2/C: now also J?.3 (Pin_3)
- net Input 2/Left: now also J?.6 (Pin_6)
Changed lines of the file:
@@
 	17150 5100 17750 5100
 Wire Wire Line
-	17750 3750 5900 3750
+	17750 3750 6850 3750
 Wire Wire Line
 	17750 5100 17750 3750
@@
 	5550 3650 2450 3650
 Wire Wire Line
-	3050 4700 5900 4700
-Wire Wire Line
-	5900 4700 5900 3750
+	3050 4700 6850 4700
+Wire Wire Line
+	6850 4700 6850 3750
 Wire Wire Line
 	3050 4700 3050 5000
@@
 	2450 3750 5500 3750
 Wire Wire Line
-	5800 4600 5800 3700
-Wire Wire Line
-	5800 3700 17850 3700
-Wire Wire Line
-	2450 4600 5800 4600
+	6800 4600 6800 3700
+Wire Wire Line
+	6800 3700 17850 3700
+Wire Wire Line
+	2450 4600 6800 4600
 Wire Wire Line
 	7700 17250 7100 17250
@@
 Wire Wire Line
 	1000 4350 8500 4350
+Wire Wire Line
+	7700 9700 8350 9700
+Wire Wire Line
+	8350 9700 8350 9150
+Wire Wire Line
+	8350 9150 5750 9150
+Wire Wire Line
+	5750 9150 5750 3850
+Wire Wire Line
+	5750 3850 2450 3850
+Wire Wire Line
+	7700 10000 8400 10000
+Wire Wire Line
+	8400 10000 8400 9100
+Wire Wire Line
+	8400 9100 5800 9100
+Wire Wire Line
+	5800 9100 5800 3450
+Wire Wire Line
+	5800 3450 2450 3450
+Wire Wire Line
+	7700 10300 8450 10300
+Wire Wire Line
+	8450 10300 8450 9050
+Wire Wire Line
+	8450 9050 5850 9050
+Wire Wire Line
+	5850 9050 5850 3250
+Wire Wire Line
+	5850 3250 900  3250
+Wire Wire Line
+	900  3250 900  3450
+Wire Wire Line
+	900  3450 1150 3450
+Wire Wire Line
+	7100 9700 -200 9700
+Wire Wire Line
+	-200 9700 -200 3950
+Wire Wire Line
+	-200 3950 1150 3950
+Wire Wire Line
+	7100 10000 -350 10000
+Wire Wire Line
+	-350 10000 -350 3650
+Wire Wire Line
+	-350 3650 1150 3650
+Wire Wire Line
+	7100 10300 -850 10300
+Wire Wire Line
+	-850 10300 -850 3550
+Wire Wire Line
+	-850 3550 1150 3550
 $EndSCHEMATC

Commit message: Finished wiring switch 2
Connections:
- net Input 1/Blue: now also J?.9 (Pin_9)
- net Input 1/Composite: now also J?.6 (Pin_6)
- net Input 1/Green: now also J?.3 (Pin_3)
- net Input 1/Red: now also J?.6 (Pin_6)
- net Input 1/Right: now also J?.9 (Pin_9)
- net Input 1/Y: now also J?.3 (Pin_3)
Changed lines of the file:
@@
 	24300 5950 24550 5950
 Wire Wire Line
-	4600 5300 4050 5300
+	4250 5300 4050 5300
 NoConn ~ 30500 5500
 NoConn ~ 29900 5500
@@
 	7000 9600 7100 9600
 Wire Wire Line
-	7050 4750 7050 4450
-Wire Wire Line
-	7050 4450 3250 4450
-Wire Wire Line
-	3250 4450 3250 5000
+	3250 4750 3250 5000
 Wire Wire Line
 	3250 5000 3450 5000
@@
 	28350 6450 28350 17650
 Wire Wire Line
-	4600 7950 4600 5300
+	4250 7950 4250 5300
 Wire Wire Line
 	24550 6300 24550 7950
@@
 Wire Wire Line
 	10400 1150 10400 4550
-Wire Wire Line
-	7300 4750 7050 4750
 Wire Wire Line
 	7950 5000 8100 5000
@@
 $EndComp
 Wire Wire Line
-	18050 3450 8500 3450
+	18050 3450 9300 3450
 Wire Wire Line
 	18050 5700 18050 3450
@@
 	17150 5100 17750 5100
 Wire Wire Line
-	17750 3750 6850 3750
+	17750 3750 9500 3750
 Wire Wire Line
 	17750 5100 17750 3750
@@
 	26350 6800 26250 6800
 Wire Wire Line
-	24550 7950 4600 7950
+	24550 7950 4250 7950
 Wire Wire Line
 	11250 4450 29600 4450
@@
 	15100 5100 15100 5700
 Wire Wire Line
-	15100 5700 7400 5700
-Wire Wire Line
-	7400 5700 7400 6350
-Wire Wire Line
-	7400 6350 850  6350
+	15100 5700 8100 5700
+Wire Wire Line
+	8100 5700 8100 6350
+Wire Wire Line
+	8100 6350 850  6350
 Wire Wire Line
 	850  6350 850  5100
@@
 	14000 6150 14200 6150
 Wire Wire Line
-	13400 6400 5950 6400
-Wire Wire Line
-	5950 6400 5950 10200
-Wire Wire Line
-	5950 10200 7100 10200
+	13400 6400 6450 6400
+Wire Wire Line
+	6450 6400 6450 10200
+Wire Wire Line
+	6450 10200 7100 10200
 $Comp
 L Jumper:Jumper_2_Bridged J20
@@
 	9100 16650 9100 14450
 Wire Wire Line
-	9100 14450 5400 14450
-Wire Wire Line
-	5400 14450 5400 4050
-Wire Wire Line
-	5400 4050 2450 4050
+	9100 14450 5900 14450
+Wire Wire Line
+	5900 14450 5900 4050
+Wire Wire Line
+	5900 4050 2450 4050
 Wire Wire Line
 	8300 16950 9150 16950
@@
 	9150 16950 9150 14400
 Wire Wire Line
-	9150 14400 5450 14400
-Wire Wire Line
-	5450 14400 5450 3950
-Wire Wire Line
-	5450 3950 2450 3950
+	9150 14400 5950 14400
+Wire Wire Line
+	5950 14400 5950 3950
+Wire Wire Line
+	5950 3950 2450 3950
 Wire Wire Line
 	8300 17250 9050 17250
@@
 	9050 17250 9050 14600
 Wire Wire Line
-	9050 14600 5350 14600
-Wire Wire Line
-	5350 14600 5350 4150
-Wire Wire Line
-	5350 4150 2450 4150
+	9050 14600 5850 14600
+Wire Wire Line
+	5850 14600 5850 4150
+Wire Wire Line
+	5850 4150 2450 4150
 Wire Wire Line
 	7700 16650 7300 16650
@@
 	7300 16650 7300 14300
 Wire Wire Line
-	7300 14300 5500 14300
-Wire Wire Line
-	5500 14300 5500 3750
+	7300 14300 6000 14300
+Wire Wire Line
+	6000 14300 6000 3750
 Wire Wire Line
 	7700 16950 7150 16950
@@
 	7150 16950 7150 14200
 Wire Wire Line
-	7150 14200 5550 14200
-Wire Wire Line
-	5550 14200 5550 3650
-Wire Wire Line
-	5550 3650 2450 3650
-Wire Wire Line
-	3050 4700 6850 4700
-Wire Wire Line
-	6850 4700 6850 3750
+	7150 14200 6050 14200
+Wire Wire Line
+	6050 14200 6050 3650
+Wire Wire Line
+	6050 3650 2450 3650
+Wire Wire Line
+	3050 4700 9500 4700
+Wire Wire Line
+	9500 4700 9500 3750
 Wire Wire Line
 	3050 4700 3050 5000
 Wire Wire Line
-	2450 3750 5500 3750
-Wire Wire Line
-	6800 4600 6800 3700
-Wire Wire Line
-	6800 3700 17850 3700
-Wire Wire Line
-	2450 4600 6800 4600
+	2450 3750 6000 3750
+Wire Wire Line
+	9400 4600 9400 3700
+Wire Wire Line
+	9400 3700 17850 3700
+Wire Wire Line
+	2450 4600 9400 4600
 Wire Wire Line
 	7700 17250 7100 17250
@@
 	7100 17250 7100 14150
 Wire Wire Line
-	7100 14150 5650 14150
-Wire Wire Line
-	5650 14150 5650 3550
-Wire Wire Line
-	5650 3550 2450 3550
-Wire Wire Line
-	8500 4350 8500 3450
-Wire Wire Line
-	1000 4350 8500 4350
+	7100 14150 6150 14150
+Wire Wire Line
+	6150 14150 6150 3550
+Wire Wire Line
+	6150 3550 2450 3550
+Wire Wire Line
+	9300 4350 9300 3450
+Wire Wire Line
+	1000 4350 9300 4350
 Wire Wire Line
 	7700 9700 8350 9700
@@
 	8350 9700 8350 9150
 Wire Wire Line
-	8350 9150 5750 9150
-Wire Wire Line
-	5750 9150 5750 3850
-Wire Wire Line
-	5750 3850 2450 3850
+	8350 9150 6250 9150
+Wire Wire Line
+	6250 9150 6250 3850
+Wire Wire Line
+	6250 3850 2450 3850
 Wire Wire Line
 	7700 10000 8400 10000
@@
 	8400 10000 8400 9100
 Wire Wire Line
-	8400 9100 5800 9100
-Wire Wire Line
-	5800 9100 5800 3450
-Wire Wire Line
-	5800 3450 2450 3450
+	8400 9100 6300 9100
+Wire Wire Line
+	6300 9100 6300 3450
+Wire Wire Line
+	6300 3450 2450 3450
 Wire Wire Line
 	7700 10300 8450 10300
@@
 	8450 10300 8450 9050
 Wire Wire Line
-	8450 9050 5850 9050
-Wire Wire Line
-	5850 9050 5850 3250
-Wire Wire Line
-	5850 3250 900  3250
+	8450 9050 6350 9050
+Wire Wire Line
+	6350 9050 6350 3250
+Wire Wire Line
+	6350 3250 900  3250
 Wire Wire Line
 	900  3250 900  3450
@@
 Wire Wire Line
 	-850 3550 1150 3550
+Wire Wire Line
+	4900 16400 5050 16400
+Wire Wire Line
+	5050 2900 2450 2900
+Wire Wire Line
+	5050 2900 5050 16400
+Wire Wire Line
+	3250 4750 7300 4750
+Wire Wire Line
+	4900 16700 5100 16700
+Wire Wire Line
+	5100 16700 5100 2800
+Wire Wire Line
+	5100 2800 2450 2800
+Wire Wire Line
+	4900 17000 5150 17000
+Wire Wire Line
+	5150 17000 5150 3000
+Wire Wire Line
+	5150 3000 2450 3000
+Wire Wire Line
+	4300 16400 4100 16400
+Wire Wire Line
+	4100 16400 4100 15900
+Wire Wire Line
+	4100 15900 5000 15900
+Wire Wire Line
+	5000 15900 5000 2600
+Wire Wire Line
+	5000 2600 2450 2600
+Wire Wire Line
+	4300 16700 4050 16700
+Wire Wire Line
+	4050 16700 4050 15850
+Wire Wire Line
+	4050 15850 4950 15850
+Wire Wire Line
+	4950 15850 4950 2500
+Wire Wire Line
+	4950 2500 2450 2500
+Wire Wire Line
+	4300 17000 4000 17000
+Wire Wire Line
+	4000 17000 4000 15800
+Wire Wire Line
+	4000 15800 4900 15800
+Wire Wire Line
+	4900 15800 4900 2400
+Wire Wire Line
+	4900 2400 2450 2400
 $EndSCHEMATC

Commit message: Finished wiring switch 1
Connections:
- net Input 1/1: now also J?.9 (Pin_9)
- net Input 1/2: now also J?.9 (Pin_9)
- net Input 1/3: now also J?.6 (Pin_6)
- net Input 1/6: now also J?.3 (Pin_3)
- net Input 1/C: now also J?.3 (Pin_3)
- net Input 1/Left: now also J?.6 (Pin_6)
Other:
- moved on the sheet: J?
Changed lines of the file:
@@
 L Connector_Generic:Conn_01x09 J?
 U 1 1 60FBB208
-P 3650 5300
-F 0 "J?" H 3600 5850 50  0000 L CNN
-F 1 "SW1_L" H 3450 4750 50  0000 L CNN
-F 2 "" H 3650 5300 50  0001 C CNN
-F 3 "~" H 3650 5300 50  0001 C CNN
-	1    3650 5300
+P 3650 11500
+F 0 "J?" H 3600 12050 50  0000 L CNN
+F 1 "SW1_L" H 3450 10950 50  0000 L CNN
+F 2 "" H 3650 11500 50  0001 C CNN
+F 3 "~" H 3650 11500 50  0001 C CNN
+	1    3650 11500
 	1    0    0    -1
 $EndComp
@@
 L Connector_Generic:Conn_01x09 J?
 U 1 1 60FBB70F
-P 3850 5300
-F 0 "J?" H 3800 5850 50  0000 L CNN
-F 1 "SW1_R" H 3650 4750 50  0000 L CNN
-F 2 "" H 3850 5300 50  0001 C CNN
-F 3 "~" H 3850 5300 50  0001 C CNN
-	1    3850 5300
+P 3850 11500
+F 0 "J?" H 3800 12050 50  0000 L CNN
+F 1 "SW1_R" H 3650 10950 50  0000 L CNN
+F 2 "" H 3850 11500 50  0001 C CNN
+F 3 "~" H 3850 11500 50  0001 C CNN
+	1    3850 11500
 	-1   0    0    -1
 $EndComp
@@
 Wire Wire Line
 	24300 5950 24550 5950
-Wire Wire Line
-	4250 5300 4050 5300
 NoConn ~ 30500 5500
 NoConn ~ 29900 5500
@@
 	26800 5750 26950 5750
 Wire Wire Line
-	4300 8350 4300 5000
-Wire Wire Line
-	4300 5000 4050 5000
-Wire Wire Line
 	29400 5000 29400 3400
 Wire Wire Line
@@
 	27600 5650 27600 8400
 Wire Wire Line
-	27600 8400 3850 8450
-Wire Wire Line
-	3850 8450 3850 16300
+	27600 8400 22950 8400
 Wire Wire Line
 	3850 16300 4300 16300
@@
 NoConn ~ 7100 10100
 NoConn ~ 7700 10100
-NoConn ~ 3450 4900
-NoConn ~ 4050 4900
-NoConn ~ 4050 5200
-NoConn ~ 3450 5200
-NoConn ~ 3450 5500
-NoConn ~ 4050 5500
+NoConn ~ 3450 11100
+NoConn ~ 4050 11100
+NoConn ~ 4050 11400
+NoConn ~ 3450 11400
+NoConn ~ 3450 11700
+NoConn ~ 4050 11700
 $Comp
 L Jumper:Jumper_2_Bridged J14
@@
 	35100 15800 35100 21100
 Wire Wire Line
-	35100 21100 2100 21100
-Wire Wire Line
-	2100 21100 2100 8300
-Wire Wire Line
-	2100 8300 3000 8300
-Wire Wire Line
-	3000 8300 3000 5200
-Wire Wire Line
-	3000 5200 2450 5200
+	35100 21100 2750 21100
+Wire Wire Line
+	2750 5200 2450 5200
 Wire Wire Line
 	26650 16100 34950 16100
@@
 	34950 16100 34950 20900
 Wire Wire Line
-	34950 20900 2350 20900
-Wire Wire Line
-	2350 20900 2350 8600
-Wire Wire Line
-	2350 8600 3100 8600
-Wire Wire Line
-	3100 8600 3100 5100
-Wire Wire Line
-	3100 5100 2450 5100
-Wire Wire Line
-	2450 5300 2900 5300
-Wire Wire Line
-	2900 5300 2900 8250
-Wire Wire Line
-	1650 8250 1650 21500
-Wire Wire Line
-	1650 21500 34750 21500
+	34950 20900 2800 20900
+Wire Wire Line
+	2800 5100 2450 5100
+Wire Wire Line
+	2450 5300 2700 5300
+Wire Wire Line
+	2700 21500 34750 21500
 Wire Wire Line
 	34750 21500 34750 16400
-Wire Wire Line
-	1650 8250 2900 8250
 $Comp
 L Jumper:Jumper_2_Bridged J16
@@
 	24100 15800 24100 19500
 Wire Wire Line
-	24100 19500 3150 19500
-Wire Wire Line
-	3150 19500 3150 4900
-Wire Wire Line
-	3150 4900 2450 4900
+	24100 19500 2850 19500
+Wire Wire Line
+	2850 19500 2850 4900
+Wire Wire Line
+	2850 4900 2450 4900
 Wire Wire Line
 	26050 16100 24300 16100
@@
 	24300 16100 24300 19650
 Wire Wire Line
-	24300 19650 2850 19650
-Wire Wire Line
-	2850 19650 2850 4800
-Wire Wire Line
-	2850 4800 2450 4800
+	24300 19650 2650 19650
+Wire Wire Line
+	2650 19650 2650 4800
+Wire Wire Line
+	2650 4800 2450 4800
 Wire Wire Line
 	26050 16400 24450 16400
@@
 	2600 4700 2450 4700
 Wire Wire Line
-	3050 5000 2450 5000
-Wire Wire Line
-	4200 7150 4200 5600
-Wire Wire Line
-	4200 5600 4050 5600
+	2900 5000 2450 5000
+Wire Wire Line
+	17200 7150 17200 11800
+Wire Wire Line
+	17200 11800 4050 11800
 Wire Wire Line
 	41900 6950 41900 3000
@@
 	7000 9600 7100 9600
 Wire Wire Line
-	3250 4750 3250 5000
-Wire Wire Line
-	3250 5000 3450 5000
-Wire Wire Line
 	28350 6450 28350 17650
-Wire Wire Line
-	4250 7950 4250 5300
-Wire Wire Line
-	24550 6300 24550 7950
 Wire Wire Line
 	24300 9900 24300 5950
@@
 	21050 6950 41900 6950
 Wire Wire Line
-	18200 7150 4200 7150
+	18200 7150 17200 7150
 Wire Wire Line
 	20650 6950 19500 6950
@@
 NoConn ~ 17150 4900
 Wire Wire Line
-	17650 8350 4300 8350
-Wire Wire Line
-	17650 5750 17650 8350
+	17650 5750 17650 11200
 Wire Wire Line
 	26400 5750 17650 5750
@@
 Wire Wire Line
 	26350 6800 26250 6800
-Wire Wire Line
-	24550 7950 4250 7950
 Wire Wire Line
 	11250 4450 29600 4450
@@
 	8000 5500 8000 6550
 Wire Wire Line
-	8000 6550 3250 6550
-Wire Wire Line
-	3250 6550 3250 5300
-Wire Wire Line
-	3250 5300 3450 5300
+	8000 6550 3200 6550
+Wire Wire Line
+	3200 6550 3200 11500
+Wire Wire Line
+	3200 11500 3450 11500
 Wire Wire Line
 	14300 5300 14300 2850
@@
 	13150 6250 13300 6250
 Wire Wire Line
-	12750 6250 3350 6250
-Wire Wire Line
-	3350 6250 3350 5600
-Wire Wire Line
-	3350 5600 3450 5600
+	12750 6250 3100 6250
+Wire Wire Line
+	3100 6250 3100 11800
+Wire Wire Line
+	3100 11800 3450 11800
 Wire Wire Line
 	12750 6050 12450 6050
@@
 	6050 3650 2450 3650
 Wire Wire Line
-	3050 4700 9500 4700
+	2900 4700 9500 4700
 Wire Wire Line
 	9500 4700 9500 3750
 Wire Wire Line
-	3050 4700 3050 5000
+	2900 4700 2900 5000
 Wire Wire Line
 	2450 3750 6000 3750
@@
 	5050 2900 5050 16400
 Wire Wire Line
-	3250 4750 7300 4750
-Wire Wire Line
 	4900 16700 5100 16700
 Wire Wire Line
@@
 Wire Wire Line
 	4900 2400 2450 2400
+Wire Wire Line
+	4850 2700 2450 2700
+Wire Wire Line
+	4050 11300 4850 11300
+Wire Wire Line
+	4850 2700 4850 11300
+Wire Wire Line
+	4050 11600 4800 11600
+Wire Wire Line
+	4800 11600 4800 2300
+Wire Wire Line
+	4800 2300 2450 2300
+Wire Wire Line
+	4050 11900 4750 11900
+Wire Wire Line
+	4750 11900 4750 2100
+Wire Wire Line
+	4750 2100 900  2100
+Wire Wire Line
+	900  2100 900  2300
+Wire Wire Line
+	900  2300 1150 2300
+Wire Wire Line
+	3850 15250 22950 15250
+Wire Wire Line
+	22950 15250 22950 8400
+Wire Wire Line
+	3850 15250 3850 16300
+Wire Wire Line
+	4050 11200 17650 11200
+Wire Wire Line
+	4050 11500 24550 11500
+Wire Wire Line
+	24550 6300 24550 11500
+Wire Wire Line
+	2700 5300 2700 21500
+Wire Wire Line
+	2750 5200 2750 21100
+Wire Wire Line
+	2800 5100 2800 20900
+Wire Wire Line
+	3450 11200 3300 11200
+Wire Wire Line
+	3300 11200 3300 4750
+Wire Wire Line
+	3300 4750 7300 4750
+Wire Wire Line
+	3450 11300 -3550 11300
+Wire Wire Line
+	-3550 11300 -3550 2800
+Wire Wire Line
+	-3550 2800 1150 2800
+Wire Wire Line
+	3450 11600 -4050 11600
+Wire Wire Line
+	-4050 11600 -4050 2500
+Wire Wire Line
+	-4050 2500 1150 2500
+Wire Wire Line
+	3450 11900 -4700 11900
+Wire Wire Line
+	-4700 11900 -4700 2400
+Wire Wire Line
+	-4700 2400 1150 2400
 $EndSCHEMATC

Commit message: Cleaning up extra ethernet pins
Setting no connects on the ports themselves and eliminating the extra
heirarchal labels and pins
Changed lines of the file:
@@
 F11 "2" U R 40100 3100 50
 F12 "3" U R 40100 3200 50
-F13 "4" U R 40100 3300 50
-F14 "5" U R 40100 3400 50
-F15 "6" U R 40100 3500 50
-F16 "7" U R 40100 3600 50
-F17 "8" U R 40100 3700 50
+F13 "6" U R 40100 3500 50
 $EndSheet
 $Sheet
@@
 F11 "2" U L 1150 3550 50
 F12 "3" U L 1150 3650 50
-F13 "4" U L 1150 3750 50
-F14 "5" U L 1150 3850 50
-F15 "6" U L 1150 3950 50
-F16 "7" U L 1150 4050 50
-F17 "8" U L 1150 4150 50
+F13 "6" U L 1150 3950 50
 $EndSheet
 $Sheet
@@
 F11 "2" U L 1150 4700 50
 F12 "3" U L 1150 4800 50
-F13 "4" U L 1150 4900 50
-F14 "5" U L 1150 5000 50
-F15 "6" U L 1150 5100 50
-F16 "7" U L 1150 5200 50
-F17 "8" U L 1150 5300 50
+F13 "6" U L 1150 5100 50
 $EndSheet
 Text Notes 32150 1950 0    50   ~ 0
@@
 F11 "2" U L 1150 2400 50
 F12 "3" U L 1150 2500 50
-F13 "4" U L 1150 2600 50
-F14 "5" U L 1150 2700 50
-F15 "6" U L 1150 2800 50
-F16 "7" U L 1150 2900 50
-F17 "8" U L 1150 3000 50
+F13 "6" U L 1150 2800 50
 $EndSheet
 Text Notes 13650 1150 0    50   ~ 0
