File: gamestop-av-switch/gamestop-av-switch.sch (KiCad schematic (older format))
At the start: 61 parts

Commit message: Annotating and satisfying ERC
Parts:
- gave numbers to parts that had none: 14
Changed lines of the file:
@@
 Switches are numbered 1-7 from left to right\nlooking at the top of the PCB\n\nPins are numbered top to bottom looking at\nbottom of PCB with connectors towards the front
 $Comp
-L Connector_Generic:Conn_01x09 J?
+L Connector_Generic:Conn_01x09 J48
 U 1 1 60FBB208
 P 3650 11500
-F 0 "J?" H 3600 12050 50  0000 L CNN
+F 0 "J48" H 3600 12050 50  0000 L CNN
 F 1 "SW1_L" H 3450 10950 50  0000 L CNN
 F 2 "" H 3650 11500 50  0001 C CNN
@@
 $EndComp
 $Comp
-L Connector_Generic:Conn_01x09 J?
+L Connector_Generic:Conn_01x09 J49
 U 1 1 60FBB70F
 P 3850 11500
-F 0 "J?" H 3800 12050 50  0000 L CNN
+F 0 "J49" H 3800 12050 50  0000 L CNN
 F 1 "SW1_R" H 3650 10950 50  0000 L CNN
 F 2 "" H 3850 11500 50  0001 C CNN
@@
 $EndComp
 $Comp
-L Connector_Generic:Conn_01x09 J?
+L Connector_Generic:Conn_01x09 J50
 U 1 1 60FBDD95
 P 4500 16600
-F 0 "J?" H 4450 17150 50  0000 L CNN
+F 0 "J50" H 4450 17150 50  0000 L CNN
 F 1 "SW2_L" H 4300 16050 50  0000 L CNN
 F 2 "" H 4500 16600 50  0001 C CNN
@@
 $EndComp
 $Comp
-L Connector_Generic:Conn_01x09 J?
+L Connector_Generic:Conn_01x09 J51
 U 1 1 60FBDD9B
 P 4700 16600
-F 0 "J?" H 4650 17150 50  0000 L CNN
+F 0 "J51" H 4650 17150 50  0000 L CNN
 F 1 "SW2_R" H 4500 16050 50  0000 L CNN
 F 2 "" H 4700 16600 50  0001 C CNN
@@
 $EndComp
 $Comp
-L Connector_Generic:Conn_01x09 J?
+L Connector_Generic:Conn_01x09 J52
 U 1 1 60FBE8B7
 P 7300 9900
-F 0 "J?" H 7250 10450 50  0000 L CNN
+F 0 "J52" H 7250 10450 50  0000 L CNN
 F 1 "SW3_L" H 7100 9350 50  0000 L CNN
 F 2 "" H 7300 9900 50  0001 C CNN
@@
 $EndComp
 $Comp
-L Connector_Generic:Conn_01x09 J?
+L Connector_Generic:Conn_01x09 J53
 U 1 1 60FBE8BD
 P 7500 9900
-F 0 "J?" H 7450 10450 50  0000 L CNN
+F 0 "J53" H 7450 10450 50  0000 L CNN
 F 1 "SW3_R" H 7300 9350 50  0000 L CNN
 F 2 "" H 7500 9900 50  0001 C CNN
@@
 $EndComp
 $Comp
-L Connector_Generic:Conn_01x09 J?
+L Connector_Generic:Conn_01x09 J54
 U 1 1 60FBEFAF
 P 7900 16850
-F 0 "J?" H 7850 17400 50  0000 L CNN
+F 0 "J54" H 7850 17400 50  0000 L CNN
 F 1 "SW4_L" H 7700 16300 50  0000 L CNN
 F 2 "" H 7900 16850 50  0001 C CNN
@@
 $EndComp
 $Comp
-L Connector_Generic:Conn_01x09 J?
+L Connector_Generic:Conn_01x09 J55
 U 1 1 60FBEFB5
 P 8100 16850
-F 0 "J?" H 8050 17400 50  0000 L CNN
+F 0 "J55" H 8050 17400 50  0000 L CNN
 F 1 "SW4_R" H 7900 16300 50  0000 L CNN
 F 2 "" H 8100 16850 50  0001 C CNN
@@
 $EndComp
 $Comp
-L Connector_Generic:Conn_01x09 J?
+L Connector_Generic:Conn_01x09 J58
 U 1 1 60FBFD53
 P 26250 16000
-F 0 "J?" H 26200 16550 50  0000 L CNN
+F 0 "J58" H 26200 16550 50  0000 L CNN
 F 1 "SW6_L" H 26050 15450 50  0000 L CNN
 F 2 "" H 26250 16000 50  0001 C CNN
@@
 $EndComp
 $Comp
-L Connector_Generic:Conn_01x09 J?
+L Connector_Generic:Conn_01x09 J59
 U 1 1 60FBFD59
 P 26450 16000
-F 0 "J?" H 26400 16550 50  0000 L CNN
+F 0 "J59" H 26400 16550 50  0000 L CNN
 F 1 "SW6_R" H 26250 15450 50  0000 L CNN
 F 2 "" H 26450 16000 50  0001 C CNN
@@
 $EndComp
 $Comp
-L Connector_Generic:Conn_01x09 J?
+L Connector_Generic:Conn_01x09 J60
 U 1 1 60FC0237
 P 30100 5300
-F 0 "J?" H 30050 5850 50  0000 L CNN
+F 0 "J60" H 30050 5850 50  0000 L CNN
 F 1 "SW7_L" H 29900 4750 50  0000 L CNN
 F 2 "" H 30100 5300 50  0001 C CNN
@@
 $EndComp
 $Comp
-L Connector_Generic:Conn_01x09 J?
+L Connector_Generic:Conn_01x09 J61
 U 1 1 60FC023D
 P 30300 5300
-F 0 "J?" H 30250 5850 50  0000 L CNN
+F 0 "J61" H 30250 5850 50  0000 L CNN
 F 1 "SW7_R" H 30100 4750 50  0000 L CNN
 F 2 "" H 30300 5300 50  0001 C CNN
@@
 	10400 4550 30750 4550
 $Comp
-L Connector_Generic:Conn_01x09 J?
+L Connector_Generic:Conn_01x09 J57
 U 1 1 60FBF895
 P 16950 5300
-F 0 "J?" H 16900 5850 50  0000 L CNN
+F 0 "J57" H 16900 5850 50  0000 L CNN
 F 1 "SW5_R" H 16750 4750 50  0000 L CNN
 F 2 "" H 16950 5300 50  0001 C CNN
@@
 $EndComp
 $Comp
-L Connector_Generic:Conn_01x09 J?
+L Connector_Generic:Conn_01x09 J56
 U 1 1 60FBF88F
 P 16750 5300
-F 0 "J?" H 16700 5850 50  0000 L CNN
+F 0 "J56" H 16700 5850 50  0000 L CNN
 F 1 "SW5_L" H 16550 4750 50  0000 L CNN
 F 2 "" H 16750 5300 50  0001 C CNN
@@
 Wire Wire Line
 	-4700 2400 1150 2400
+$Comp
+L power:GNDREF #PWR0101
+U 1 1 63C1CAC3
+P 18850 1650
+F 0 "#PWR0101" H 18850 1400 50  0001 C CNN
+F 1 "GNDREF" H 18855 1477 50  0000 C CNN
+F 2 "" H 18850 1650 50  0001 C CNN
+F 3 "" H 18850 1650 50  0001 C CNN
+	1    18850 1650
+	1    0    0    -1
+$EndComp
+$Comp
+L power:PWR_FLAG #FLG0101
+U 1 1 63C1DB37
+P 18850 1550
+F 0 "#FLG0101" H 18850 1625 50  0001 C CNN
+F 1 "PWR_FLAG" H 18850 1723 50  0000 C CNN
+F 2 "" H 18850 1550 50  0001 C CNN
+F 3 "~" H 18850 1550 50  0001 C CNN
+	1    18850 1550
+	1    0    0    -1
+$EndComp
+Wire Wire Line
+	18850 1550 18850 1650
 $EndSCHEMATC

Commit message: Cleaned up wiring
Connections:
- net Output/1: now also J21.1 (A); no longer J21.2 (B)
- net Output/3: now also J39.1 (A), J44.1 (A); no longer J39.2 (B), J44.2 (B)
- net Output/6: now also J37.1 (A), J43.1 (A); no longer J37.2 (B), J43.2 (B)
- net Output/Composite: now also J1.2 (B); no longer J1.1 (A)
- net Output/Y: now also J36.1 (A), J41.1 (A), J46.1 (A); no longer J36.2 (B), J41.2 (B), J46.2 (B)
- net at J48.2 (Pin_2): now also J37.2 (B); no longer J37.1 (A)
- net at J48.5 (Pin_5): now also J39.2 (B); no longer J39.1 (A)
- net at J48.8 (Pin_8): now also J22.2 (B); no longer J22.1 (A)
- net at J50.2 (Pin_2): now also J41.2 (B); no longer J41.1 (A)
- net at J50.5 (Pin_5): now also J34.2 (B); no longer J34.1 (A)
- net at J52.2 (Pin_2): now also J43.2 (B); no longer J43.1 (A)
- net at J52.5 (Pin_5): now also J44.2 (B); no longer J44.1 (A)
- net at J52.8 (Pin_8): now also J26.2 (B); no longer J26.1 (A)
- net at J54.2 (Pin_2): now also J46.2 (B); no longer J46.1 (A)
- net at J58.2 (Pin_2): now also J36.2 (B); no longer J36.1 (A)
- net at J17.1 (A), J33.2 (B): now also J13.1 (A); no longer J13.2 (B)
- net at J23.2 (B), J6.2 (B): now also J21.2 (B); no longer J21.1 (A)
- new net: J13.2 (B), J30.2 (B), J7.1 (A)
- new net: J1.1 (A), J34.1 (A), J7.2 (B)
- new net: J11.1 (A), J26.1 (A), J5.1 (A)
- new net: J20.2 (B), J22.1 (A), J5.2 (B)
Other:
- moved on the sheet: J1, J10, J11, J12, J13, J14, J15, J16, J17, J18, J19, J2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

Commit message: Swapped in final switch symbols and cleaned up wiring more
Parts:
- removed J48: SW1_L, symbol Connector_Generic:Conn_01x09
- removed J49: SW1_R, symbol Connector_Generic:Conn_01x09
- removed J50: SW2_L, symbol Connector_Generic:Conn_01x09
- removed J51: SW2_R, symbol Connector_Generic:Conn_01x09
- removed J52: SW3_L, symbol Connector_Generic:Conn_01x09
- removed J53: SW3_R, symbol Connector_Generic:Conn_01x09
- removed J54: SW4_L, symbol Connector_Generic:Conn_01x09
- removed J55: SW4_R, symbol Connector_Generic:Conn_01x09
- removed J56: SW5_L, symbol Connector_Generic:Conn_01x09
- removed J57: SW5_R, symbol Connector_Generic:Conn_01x09
- removed J58: SW6_L, symbol Connector_Generic:Conn_01x09
- removed J59: SW6_R, symbol Connector_Generic:Conn_01x09
- removed J60: SW7_L, symbol Connector_Generic:Conn_01x09
- removed J61: SW7_R, symbol Connector_Generic:Conn_01x09
- added S1: SW1, symbol SW-gElectroMech:6PDT
- added S2: SW2, symbol SW-gElectroMech:6PDT
- added S3: SW3, symbol SW-gElectroMech:6PDT
- added S4: SW4, symbol SW-gElectroMech:6PDT
- added S5: SW5, symbol SW-gElectroMech:6PDT
- added S6: SW6, symbol SW-gElectroMech:6PDT
- added S?: SW7, symbol SW-gElectroMech:6PDT
Connections:
- net Front Input/C: now also S?.3
- net Front Input/Composite: now also S?.18
- net Front Input/Left: now also S?.12
- net Front Input/Right: now also S?.9
- net Front Input/Y: now also S?.6
- net Input 1/1: now also S1.18
- net Input 1/2: now also S1.9
- net Input 1/3: now also S1.6
- net Input 1/6: now also S1.3
- net Input 1/Blue: now also S2.18
- net Input 1/C: now also S1.12
- net Input 1/Composite: now also S2.6
- net Input 1/Green: now also S2.12
- net Input 1/Left: now also S1.15
- net Input 1/Red: now also S2.15
- net Input 1/Right: now also S2.9
- net Input 1/Y: now also S2.3
- net Input 2/1: now also S3.18
- net Input 2/2: now also S3.9
- net Input 2/3: now also S3.6
- net Input 2/6: now also S3.3
- net Input 2/Blue: now also S4.18
- net Input 2/C: now also S3.12
- net Input 2/Composite: now also S4.6
- net Input 2/Green: now also S4.12
- net Input 2/Left: now also S3.15
- net Input 2/Red: now also S4.15
- net Input 2/Right: now also S4.9
- net Input 2/Y: now also S4.3
- net Input 3/1: now also S5.18
- net Input 3/2: now also S5.9
- net Input 3/3: now also S5.6
- net Input 3/6: now also S5.3
- net Input 3/Blue: now also S6.18
- net Input 3/C: now also S5.12
- net Input 3/Composite: now also S6.6
- net Input 3/Green: now also S6.12
- net Input 3/Left: now also S5.15
- net Input 3/Red: now also S6.15
- net Input 3/Right: now also S6.9
- net Input 3/Y: now also S6.3
- net Output/3: now also J18.2 (B), J39.2 (B), J44.2 (B); no longer J18.1 (A), J39.1 (A), J44.1 (A)
- net Output/6: now also J37.2 (B), J43.2 (B), J47.2 (B); no longer J37.1 (A), J43.1 (A), J47.1 (A)
- net Output/C: now also S?.2
- net Output/Left: now also S?.11
- net Output/Right: now also S2.8, S4.8, S6.8, S?.8
- net Output/Y: now also J36.2 (B), J41.2 (B), J46.2 (B), S?.5; no longer J36.1 (A), J41.1 (A), J46.1 (A)
- net at J22.2 (B): now also J20.2 (B), J5.2 (B)
- net at J40.1 (A): now also S1.11
- net at J38.1 (A): now also S1.14
- net at J23.1 (A): now also S1.17
- net at J34.2 (B): now also J1.1 (A), J7.2 (B)
- net at J10.2 (B), J4.1 (A): now also S2.11
- net at J25.1 (A): now also S2.14
- net at J24.1 (A): now also S2.17
- net at J26.2 (B): now also J11.2 (B), J5.1 (A)
- net at J45.1 (A): now also S3.11
- net at J42.1 (A): now also S3.14
- net at J27.1 (A): now also S3.17
- net at J30.1 (A): now also S4.5
- net at J10.1 (A), J14.2 (B): now also S4.11
- net at J28.1 (A): now also S4.14
- net at J29.1 (A): now also S4.17
- net at J32.2 (B): now also J11.1 (A)
- net at J35.1 (A): now also S5.11
- net at J19.1 (A): now also S5.14
- net at J17.2 (B): now also J13.1 (A), J33.2 (B)
- net at J14.1 (A): now also S6.11
- net at J15.1 (A): now also S6.14
- net at J16.1 (A): now also S6.17
- net at J33.1 (A): now also S?.17
- net at J32.1 (A): now also S5.8; no longer J11.2 (B)
- new net: J17.1 (A), S6.5
- new net: J34.1 (A), S2.5
- new net: J36.1 (A), S6.2
- new net: J46.1 (A), S4.2
- new net: J41.1 (A), S2.2
- new net: J47.1 (A), S5.2
- new net: J43.1 (A), S3.2
- new net: J37.1 (A), S1.2
- new net: J18.1 (A), S5.5
- new net: J44.1 (A), S3.5
- new net: J39.1 (A), S1.5
- new net: J26.1 (A), S3.8
- new net: J22.1 (A), S1.8
- new net: S?.13, S?.14, S?.15
Other:
- moved on the sheet: J1, J10, J11, J12, J13, J14, J15, J16, J17, J18, J19, J2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

Commit message: added another text note
Other:
- note added: "Switches are mechanically linked\nso depressing one pair of switches\nunpresses the other switches."
Changed lines of the file:
@@
 Wire Wire Line
 	31750 9150 41750 9150
+Text Notes 32750 2950 0    50   ~ 0
+Switches are mechanically linked\nso depressing one pair of switches\nunpresses the other switches.
 $EndSCHEMATC
