File: gamestop-av-switch/front-input.sch (KiCad schematic (older format))
At the start: 6 parts

Commit message: Annotating and satisfying ERC
Parts:
- gave numbers to parts that had none: 6
Changed lines of the file:
@@
 P 4350 3250
 AR Path="/60F42E71" Ref="J?"  Part="1"
-AR Path="/60F42772/60F42E71" Ref="J?"  Part="1"
-F 0 "J?" H 4450 3225 50  0000 L CNN
+AR Path="/60F42772/60F42E71" Ref="J63"  Part="1"
+F 0 "J63" H 4450 3225 50  0000 L CNN
 F 1 "L4" H 4450 3134 50  0000 L CNN
 F 2 "" H 4350 3250 50  0001 C CNN
@@
 P 4400 4400
 AR Path="/60F42E77" Ref="J?"  Part="1"
-AR Path="/60F42772/60F42E77" Ref="J?"  Part="1"
-F 0 "J?" H 4400 4767 50  0000 C CNN
+AR Path="/60F42772/60F42E77" Ref="J64"  Part="1"
+F 0 "J64" H 4400 4767 50  0000 C CNN
 F 1 "SV4" H 4400 4676 50  0000 C CNN
 F 2 "" H 4400 4400 50  0001 C CNN
@@
 P 3850 3250
 AR Path="/60F42E7D" Ref="J?"  Part="1"
-AR Path="/60F42772/60F42E7D" Ref="J?"  Part="1"
-F 0 "J?" H 3950 3225 50  0000 L CNN
+AR Path="/60F42772/60F42E7D" Ref="J62"  Part="1"
+F 0 "J62" H 3950 3225 50  0000 L CNN
 F 1 "Y4" H 3950 3134 50  0000 L CNN
 F 2 "" H 3850 3250 50  0001 C CNN
@@
 P 5200 3250
 AR Path="/60F433D1" Ref="J?"  Part="1"
-AR Path="/60F42772/60F433D1" Ref="J?"  Part="1"
-F 0 "J?" H 5300 3225 50  0000 L CNN
+AR Path="/60F42772/60F433D1" Ref="J65"  Part="1"
+F 0 "J65" H 5300 3225 50  0000 L CNN
 F 1 "R4" H 5300 3134 50  0000 L CNN
 F 2 "" H 5200 3250 50  0001 C CNN
@@
 $EndComp
 $Comp
-L Connector_Generic:Conn_01x06 J?
+L Connector_Generic:Conn_01x06 J66
 U 1 1 60F453E3
 P 6300 3900
-F 0 "J?" H 6380 3892 50  0000 L CNN
+F 0 "J66" H 6380 3892 50  0000 L CNN
 F 1 "Conn2" H 6380 3801 50  0000 L CNN
 F 2 "" H 6300 3900 50  0001 C CNN
@@
 $EndComp
 $Comp
-L Connector_Generic:Conn_01x06 J?
+L Connector_Generic:Conn_01x06 J67
 U 1 1 60F460D3
 P 6750 3900
-F 0 "J?" H 6668 4317 50  0000 C CNN
+F 0 "J67" H 6668 4317 50  0000 C CNN
 F 1 "Conn1" H 6668 4226 50  0000 C CNN
 F 2 "" H 6750 3900 50  0001 C CNN
@@
 	6950 3700 7200 3700
 $Comp
-L power:GNDREF #PWR?
+L power:GNDREF #PWR01
 U 1 1 60F63D72
 P 7200 4300
-F 0 "#PWR?" H 7200 4050 50  0001 C CNN
+F 0 "#PWR01" H 7200 4050 50  0001 C CNN
 F 1 "GNDREF" H 7205 4127 50  0000 C CNN
 F 2 "" H 7200 4300 50  0001 C CNN
