File: gamestop-av-switch/input-1.sch (KiCad schematic (older format))
At the start: 8 parts

Commit message: Cleaning up extra ethernet pins
Setting no connects on the ports themselves and eliminating the extra
heirarchal labels and pins
Connections:
- net 4: no longer names the net of J?.4
- net 5: no longer names the net of J?.5
- net 7: no longer names the net of J?.7
- net 8: no longer names the net of J?.8
- no-connect marks 0 -> 4
Changed lines of the file:
@@
 Text HLabel 9750 3300 2    50   UnSpc ~ 0
 3
-Text HLabel 9750 3200 2    50   UnSpc ~ 0
-4
-Text HLabel 9750 3100 2    50   UnSpc ~ 0
-5
 Text HLabel 9750 3000 2    50   UnSpc ~ 0
 6
-Text HLabel 9750 2900 2    50   UnSpc ~ 0
-7
-Text HLabel 9750 2800 2    50   UnSpc ~ 0
-8
-Wire Wire Line
-	9450 2800 9750 2800
-Wire Wire Line
-	9450 2900 9750 2900
 Wire Wire Line
 	9450 3000 9750 3000
-Wire Wire Line
-	9450 3100 9750 3100
-Wire Wire Line
-	9450 3200 9750 3200
 Wire Wire Line
 	9450 3300 9750 3300
@@
 Wire Wire Line
 	9050 3800 9050 3700
+NoConn ~ 9450 2800
+NoConn ~ 9450 2900
+NoConn ~ 9450 3100
+NoConn ~ 9450 3200
 $EndSCHEMATC

Commit message: Annotating and satisfying ERC
Parts:
- gave numbers to parts that had none: 8
Changed lines of the file:
@@
 P 4650 3100
 AR Path="/60F651D4" Ref="J?"  Part="1"
-AR Path="/60F3FEDE/60F651D4" Ref="J?"  Part="1"
+AR Path="/60F3FEDE/60F651D4" Ref="J98"  Part="1"
 AR Path="/60F422FE/60F651D4" Ref="J?"  Part="1"
 AR Path="/60F4248B/60F651D4" Ref="J?"  Part="1"
-F 0 "J?" H 4750 3075 50  0000 L CNN
+F 0 "J98" H 4750 3075 50  0000 L CNN
 F 1 "RD1" H 4750 2984 50  0000 L CNN
 F 2 "" H 4650 3100 50  0001 C CNN
@@
 P 7050 3350
 AR Path="/60F651D5" Ref="J?"  Part="1"
-AR Path="/60F3FEDE/60F651D5" Ref="J?"  Part="1"
+AR Path="/60F3FEDE/60F651D5" Ref="J100"  Part="1"
 AR Path="/60F422FE/60F651D5" Ref="J?"  Part="1"
 AR Path="/60F4248B/60F651D5" Ref="J?"  Part="1"
-F 0 "J?" H 7050 3717 50  0000 C CNN
+F 0 "J100" H 7050 3717 50  0000 C CNN
 F 1 "SV1" H 7050 3626 50  0000 C CNN
 F 2 "" H 7050 3350 50  0001 C CNN
@@
 P 9050 3200
 AR Path="/60F65215" Ref="J?"  Part="1"
-AR Path="/60F3FEDE/60F65215" Ref="J?"  Part="1"
+AR Path="/60F3FEDE/60F65215" Ref="J101"  Part="1"
 AR Path="/60F422FE/60F65215" Ref="J?"  Part="1"
 AR Path="/60F4248B/60F65215" Ref="J?"  Part="1"
-F 0 "J?" H 9107 3867 50  0000 C CNN
+F 0 "J101" H 9107 3867 50  0000 C CNN
 F 1 "LAN1" H 9107 3776 50  0000 C CNN
 F 2 "" V 9050 3225 50  0001 C CNN
@@
 P 4650 3550
 AR Path="/60F65216" Ref="J?"  Part="1"
-AR Path="/60F3FEDE/60F65216" Ref="J?"  Part="1"
+AR Path="/60F3FEDE/60F65216" Ref="J99"  Part="1"
 AR Path="/60F422FE/60F65216" Ref="J?"  Part="1"
 AR Path="/60F4248B/60F65216" Ref="J?"  Part="1"
-F 0 "J?" H 4750 3525 50  0000 L CNN
+F 0 "J99" H 4750 3525 50  0000 L CNN
 F 1 "G1" H 4750 3434 50  0000 L CNN
 F 2 "" H 4650 3550 50  0001 C CNN
@@
 P 3400 3100
 AR Path="/60F65217" Ref="J?"  Part="1"
-AR Path="/60F3FEDE/60F65217" Ref="J?"  Part="1"
+AR Path="/60F3FEDE/60F65217" Ref="J96"  Part="1"
 AR Path="/60F422FE/60F65217" Ref="J?"  Part="1"
 AR Path="/60F4248B/60F65217" Ref="J?"  Part="1"
-F 0 "J?" H 3500 3075 50  0000 L CNN
+F 0 "J96" H 3500 3075 50  0000 L CNN
 F 1 "B1" H 3500 2984 50  0000 L CNN
 F 2 "" H 3400 3100 50  0001 C CNN
@@
 P 3400 3550
 AR Path="/60F41BCB" Ref="J?"  Part="1"
-AR Path="/60F3FEDE/60F41BCB" Ref="J?"  Part="1"
+AR Path="/60F3FEDE/60F41BCB" Ref="J97"  Part="1"
 AR Path="/60F422FE/60F41BCB" Ref="J?"  Part="1"
 AR Path="/60F4248B/60F41BCB" Ref="J?"  Part="1"
-F 0 "J?" H 3500 3525 50  0000 L CNN
+F 0 "J97" H 3500 3525 50  0000 L CNN
 F 1 "Y1" H 3500 3434 50  0000 L CNN
 F 2 "" H 3400 3550 50  0001 C CNN
@@
 P 2300 3100
 AR Path="/60F651DA" Ref="J?"  Part="1"
-AR Path="/60F3FEDE/60F651DA" Ref="J?"  Part="1"
+AR Path="/60F3FEDE/60F651DA" Ref="J94"  Part="1"
 AR Path="/60F422FE/60F651DA" Ref="J?"  Part="1"
 AR Path="/60F4248B/60F651DA" Ref="J?"  Part="1"
-F 0 "J?" H 2400 3075 50  0000 L CNN
+F 0 "J94" H 2400 3075 50  0000 L CNN
 F 1 "R1" H 2400 2984 50  0000 L CNN
 F 2 "" H 2300 3100 50  0001 C CNN
@@
 P 2300 3550
 AR Path="/60F41BD7" Ref="J?"  Part="1"
-AR Path="/60F3FEDE/60F41BD7" Ref="J?"  Part="1"
+AR Path="/60F3FEDE/60F41BD7" Ref="J95"  Part="1"
 AR Path="/60F422FE/60F41BD7" Ref="J?"  Part="1"
 AR Path="/60F4248B/60F41BD7" Ref="J?"  Part="1"
-F 0 "J?" H 2400 3525 50  0000 L CNN
+F 0 "J95" H 2400 3525 50  0000 L CNN
 F 1 "L1" H 2400 3434 50  0000 L CNN
 F 2 "" H 2300 3550 50  0001 C CNN
@@
 C
 $Comp
-L power:GNDREF #PWR?
+L power:GNDREF #PWR011
 U 1 1 60F67562
 P 5050 4050
-F 0 "#PWR?" H 5050 3800 50  0001 C CNN
+F 0 "#PWR011" H 5050 3800 50  0001 C CNN
 F 1 "GNDREF" H 5055 3877 50  0000 C CNN
 F 2 "" H 5050 4050 50  0001 C CNN
@@
 Connection ~ 7050 3750
 $Comp
-L power:GNDREF #PWR?
+L power:GNDREF #PWR012
 U 1 1 60F85B66
 P 6650 3900
-F 0 "#PWR?" H 6650 3650 50  0001 C CNN
+F 0 "#PWR012" H 6650 3650 50  0001 C CNN
 F 1 "GNDREF" H 6655 3727 50  0000 C CNN
 F 2 "" H 6650 3900 50  0001 C CNN
@@
 	9450 3500 9750 3500
 $Comp
-L power:GNDREF #PWR?
+L power:GNDREF #PWR013
 U 1 1 60F9006C
 P 9050 3800
-F 0 "#PWR?" H 9050 3550 50  0001 C CNN
+F 0 "#PWR013" H 9050 3550 50  0001 C CNN
 F 1 "GNDREF" H 9055 3627 50  0000 C CNN
 F 2 "" H 9050 3800 50  0001 C CNN
