File: gamestop-av-switch/gamestop-av-switch-no-jumpers/gamestop-av-switch.sch (KiCad schematic (older format))
At the start: 7 parts

Commit message: Final cleanup and orginization
Parts:
- gave numbers to parts that had none: 1
Connections:
- net Output/1 renamed Out_TD+
- net Output/2 renamed Out_TD-
- net Output/3 renamed Out_RD+
- net Output/6 renamed Out_RD-
- net Output/Blue renamed Out_Blue
- net Output/C renamed Out_C
- net Output/Composite renamed Out_Composite
- net Output/Green renamed Out_Green
- net Output/Left renamed Out_Left
- net Output/Red renamed Out_Red
- net Output/Right renamed Out_Right
- net Output/Y renamed Out_Y
Other:
- note added: "Switches are numbered 1-7 from left to right\nlooking at the top of the PCB\n\nPins are numbered top to bottom looking at\nbottom of PCB with connectors towards the front\n\nSee Pictures in Readme"
- note removed: "Switches are numbered 1-7 from left to right\nlooking at the top of the PCB\n\nPins are numbered top to bottom looking at\nbottom of PCB with connectors towards the front"
- moved on the sheet: S1, S2, S3, S4, S5, S6, S7
