File: advent-powered-speaker/main_pcb/main_pcb.kicad_sch (KiCad schematic)
At the start: 95 parts, among them J1 wire, J10 wire, J11 wire, J12 wire, J13 wire, J14 wire, J15 wire, J16 wire, J17 wire, J20 wire, J21 wire, J22 wire, J9 wire, Q1 C546B, Q13 C33740, Q14 C556B, Q18 C33740, Q2 C32740, Q4 C546(8)B, Q5 C32740, Q6 C546B, Q7 C546B, U1 4558DD JRC 4117B, U2 45560 JRC 4032A

Commit message: Advent Speaker complete except for some ref-des
Parts:
- removed C25: 100uF 35V, symbol Device:C_Polarized
- removed Q?: Conn_01x03, symbol Connector_Generic:Conn_01x03
- added C10, C12: 10uF 35V, symbol Device:C_Polarized
- added C13: 332J Film, symbol Device:C
- added C14: 223J Film, symbol Device:C
- added C15: 184J Film, symbol Device:C
- added C26: 4.7uF 50V, symbol Device:C_Polarized
- added C30: 684J 100V Film, symbol Device:C
- added C4: 224J Film, symbol Device:C
- added C5: 123J Film, symbol Device:C
- added C8: 224, symbol Device:C
- added D10, D11, D5: 148, symbol Device:D
- added D12, D3, D4: 1N4, symbol Device:D
- added D13: D, symbol Device:D
- added D6, D8: 48, symbol Device:D
- added J18, J8: wire, symbol Jumper:Jumper_2_Bridged
- added Q10, Q11: C546B, symbol Connector_Generic:Conn_01x03
- added Q12, Q8, Q9: C556B, symbol Connector_Generic:Conn_01x03
- added R1, R18, R24: 2k2 Ω ± 5% 0.25 W, symbol Device:R
- added R10: 470k Ω ± 5% 0.25 W, symbol Device:R
- added R11, R2, R5: 150 Ω ± 5% 0.25 W, symbol Device:R
- added R12, R20: 33k Ω ± 5% 0.25 W, symbol Device:R
- added R15: 470 Ω ± 5% 0.25 W, symbol Device:R
- added R16: 560k Ω ± 5% 0.25 W, symbol Device:R
- added R17: 10M Ω ± 5% 0.25 W, symbol Device:R
- added R21, R33: 330k Ω ± 5% 0.25 W, symbol Device:R
- added R25: T15A20K T NOBLE, symbol Device:R_Potentiometer
- added R26: 47k Ω ± 5% 0.25 W, symbol Device:R
- added R27: 1k2 Ω ± 5% 0.25 W, symbol Device:R
- added R28, R31: T15C20K T NOBLE, symbol Device:R_Potentiometer
- added R29: 510 Ω ± 2% 0.25 W, symbol Device:R
- added R30: 2k4 Ω ± 5% 0.25 W, symbol Device:R
- added R32: 1k Ω ± 5% 0.25 W, symbol Device:R
- added R34, R41, R42: 4k7 Ω ± 5% 0.25 W, symbol Device:R
- added R36, R39: 100 Ω ± 5% 0.25 W, symbol Device:R
- added R49: 150k Ω ± 5% 0.25 W, symbol Device:R
- added R60: 1k Ω ± 2% 0.25 W, symbol Device:R
- added R67: 27k Ω ± 5% 0.25 W, symbol Device:R
- added R69: 5k6 Ω ± 5% 0.25 W, symbol Device:R
- added R7: 100k Ω ± 5% 0.25 W, symbol Device:R
- gave numbers to parts that had none: 1
Connections:
- net at R43.2, R44.1: now also C25.1
- net at C6.1, C9.2, D7.2 (A)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: now also R14.2; no longer R14.1
- net at C6.2: now also C30.2, R1.1
- net at R40.2: now also Q4.3 (Pin_3), R39.1
- net at Q?.B, R58.1: now also Q5.1 (Pin_1)
- net at J20.1 (A), R19.2, U1.8 (Pin_8)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: now also C11.1, R22.1, Q9.3 (Pin_3), R17.2; no longer C11.2, R22.2
- net at U2.1 (Pin_1): now also R5.2
- net at U2.3 (Pin_3): now also A.2 (B), C27.1, R47.2, R48.2, J18.1 (A), R26.1, R67.1
- net at U2.5 (Pin_5): now also C30.1, R67.2
- net at U2.6 (Pin_6): now also R46.2, R60.1
- net at U2.7 (Pin_7): now also R2.1
- net at R68.2: now also U1.3 (Pin_3), C8.1, R7.2
- net at C21.1: now also R60.2
- net at U1.1 (Pin_1): now also R10.1, R12.2
- net at U1.2 (Pin_2): now also R10.2, R11.2
- net at U1.5 (Pin_5): now also C4.1, R26.2
- net at U1.6 (Pin_6): now also R31.2, R33.1, R69.1
- net at U1.7 (Pin_7): now also R1.2, R29.1, R32.2, R33.2
- net at R19.1: now also J?.2 (Pin_2), R18.2
- net at C?.2: now also C18.2
- net at R52.2: now also Q?.E, R38.2
- net at Q18.2 (Pin_2): now also Q14.1 (Pin_1), R56.2
- net at C9.1: now also R11.1
- net at Q?.B, R38.1: now also Q13.3 (Pin_3)
- net at Q6.2 (Pin_2): now also D5.2 (A), R42.2, R5.1
- net at D7.1 (K): now also Q7.2 (Pin_2), R14.1, C10.2
- net at J?.5 (Pin_5): now also C12.2, J8.2 (B), Q10.3 (Pin_3), Q11.3 (Pin_3), R21.1, R25.1
- net at J?.6 (Pin_6): now also R24.2, R49.2
- net at C25.2, J12.1 (A), J21.2 (B): now also R41.1
- net at C24.1: now also R36.2, R39.2
- net at J9.2 (B): now also J8.1 (A)
- net at R35.1: now also D12.1 (K), Q12.2 (Pin_2)
- net at R37.2: now also Q12.3 (Pin_3), R36.1
- net at Q13.2 (Pin_2): now also R57.2, Q12.1 (Pin_1)
- net at A.1 (A): now also C26.2
- net at Q7.1 (Pin_1): now also R15.1
- net at Q14.2 (Pin_2): now also D11.1 (K), R41.2
- net at Q4.2 (Pin_2): now also D3.2 (A), R2.2, R34.1
- net at R13.2: now also C10.1, R12.1
- new net: C12.1, D13.1 (K), R20.2, R21.2
- new net: C5.2, R30.1
- new net: C26.1, R27.2, R30.2
- new net: D6.1 (K), R18.1
- new net: C4.2, Q11.1 (Pin_1), R25.2
- new net: R24.1, R25.3
- new net: C15.1, R28.1, R29.2
- new net: C14.1, C15.2, R28.2, R69.2
- new net: C14.2, R27.1, R28.3
- new net: D12.2 (A), D4.1 (K)
- new net: D6.2 (A), D8.2 (A), Q8.1 (Pin_1), Q9.1 (Pin_1), R20.1
- new net: C11.2, R15.2, R16.1
- new net: C8.2, R49.1
- new net: Q8.2 (Pin_2), R16.2, R17.1
- new net: Q8.3 (Pin_3), Q9.2 (Pin_2)
- new net: Q10.1 (Pin_1), Q11.2 (Pin_2), R22.2
- new net: C5.1, R31.1
- new net: C13.1, R31.3
- new net: D10.1 (K), D11.2 (A)
- new net: D10.2 (A), D5.1 (K)
- new net: J18.2 (B), R7.1
- new net: D8.1 (K), R34.2, R42.1
- new net: D3.1 (K), D4.2 (A)
- new net: D13.2 (A), Q10.2 (Pin_2)
- new net: C13.2, R32.1
Other:
- note added: "Pin assignments assume white stripe is pin 1"
- moved on the sheet: C11, C21, C24, C25, C9, D7, J10, J11, J21, J?, Q7, R13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

Commit message: Updated reference designators hidden behind transistor mounting plate
Parts:
- gave numbers to parts that had none: 5
Changed lines of the file:
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@@
 		(dnp no)
 		(fields_autoplaced yes)
-		(property "Reference" "Q?"
+		(property "Reference" "Q16"
 			(at 415.29 377.1899 0)
 			(show_name no)
@@
 			(project "main_pcb"
 				(path "/59986deb-8fca-4720-9445-aa41ddfde149"
-					(reference "Q?")
+					(reference "Q16")
 					(unit 1)
 				)
@@
 		(dnp no)
 		(fields_autoplaced yes)
-		(property "Reference" "C?"
+		(property "Reference" "C17"
 			(at 709.93 542.29 90)
 			(show_name no)
@@
 			(project "main_pcb"
 				(path "/59986deb-8fca-4720-9445-aa41ddfde149"
-					(reference "C?")
+					(reference "C17")
 					(unit 1)
 				)
@@
 		(dnp no)
 		(fields_autoplaced yes)
-		(property "Reference" "Q?"
+		(property "Reference" "Q15"
 			(at 680.72 518.1599 0)
 			(show_name no)
@@
 			(project "main_pcb"
 				(path "/59986deb-8fca-4720-9445-aa41ddfde149"
-					(reference "Q?")
+					(reference "Q15")
 					(unit 1)
 				)
@@
 		(dnp no)
 		(fields_autoplaced yes)
-		(property "Reference" "Q?"
+		(property "Reference" "Q3"
 			(at 599.44 482.5999 0)
 			(show_name no)
@@
 			(project "main_pcb"
 				(path "/59986deb-8fca-4720-9445-aa41ddfde149"
-					(reference "Q?")
+					(reference "Q3")
 					(unit 1)
 				)
@@
 		(dnp no)
 		(fields_autoplaced yes)
-		(property "Reference" "Q?"
+		(property "Reference" "Q17"
 			(at 443.23 393.6999 0)
 			(show_name no)
@@
 			(project "main_pcb"
 				(path "/59986deb-8fca-4720-9445-aa41ddfde149"
-					(reference "Q?")
+					(reference "Q17")
 					(unit 1)
 				)

Commit message: fixing reference designators that were not compatible with KiCAD
Parts:
- EXT3: renamed from BASE_NEG; value Conn_01x01 -> BASE_NEG
- EXT4: renamed from TREB_NEG; value Conn_01x01 -> TREB_NEG
- EXT5: renamed from TREB_POS; value Conn_01x01 -> TREB_POS
- EXT6: renamed from BASE_POS; value Conn_01x01 -> BASE_POS
- J30: renamed from A; value wire -> A
- gave numbers to parts that had none: 3
- renumbered FUSE to F1
Changed lines of the file:
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@@
 		(dnp no)
 		(fields_autoplaced yes)
-		(property "Reference" "BASE_NEG"
+		(property "Reference" "EXT3"
 			(at 438.15 495.2999 0)
 			(show_name no)
@@
 			)
 		)
-		(property "Value" "Conn_01x01"
+		(property "Value" "BASE_NEG"
 			(at 438.15 497.8399 0)
 			(show_name no)
@@
 			(project "main_pcb"
 				(path "/59986deb-8fca-4720-9445-aa41ddfde149"
-					(reference "BASE_NEG")
+					(reference "EXT3")
 					(unit 1)
 				)
@@
 		(dnp no)
 		(fields_autoplaced yes)
-		(property "Reference" "BASE_POS"
+		(property "Reference" "EXT6"
 			(at 721.36 645.1599 0)
 			(show_name no)
@@
 			)
 		)
-		(property "Value" "Conn_01x01"
+		(property "Value" "BASE_POS"
 			(at 721.36 647.6999 0)
 			(show_name no)
@@
 			(project "main_pcb"
 				(path "/59986deb-8fca-4720-9445-aa41ddfde149"
-					(reference "BASE_POS")
+					(reference "EXT6")
 					(unit 1)
 				)
@@
 		(dnp no)
 		(fields_autoplaced yes)
-		(property "Reference" "TREB_NEG"
+		(property "Reference" "EXT4"
 			(at 438.15 507.9999 0)
 			(show_name no)
@@
 			)
 		)
-		(property "Value" "Conn_01x01"
+		(property "Value" "TREB_NEG"
 			(at 438.15 510.5399 0)
 			(show_name no)
@@
 			(project "main_pcb"
 				(path "/59986deb-8fca-4720-9445-aa41ddfde149"
-					(reference "TREB_NEG")
+					(reference "EXT4")
 					(unit 1)
 				)
@@
 		(dnp no)
 		(fields_autoplaced yes)
-		(property "Reference" "J?"
+		(property "Reference" "EXT1"
 			(at 791.21 488.95 0)
 			(show_name no)
@@
 			(project "main_pcb"
 				(path "/59986deb-8fca-4720-9445-aa41ddfde149"
-					(reference "J?")
+					(reference "EXT1")
 					(unit 1)
 				)
@@
 		(dnp no)
 		(fields_autoplaced yes)
-		(property "Reference" "H?"
+		(property "Reference" "H1"
 			(at 463.55 311.15 90)
 			(show_name no)
@@
 			(project "main_pcb"
 				(path "/59986deb-8fca-4720-9445-aa41ddfde149"
-					(reference "H?")
+					(reference "H1")
 					(unit 1)
 				)
@@
 		(dnp no)
 		(fields_autoplaced yes)
-		(property "Reference" "FUSE"
+		(property "Reference" "F1"
 			(at 449.58 274.32 90)
 			(show_name no)
@@
 			(project "main_pcb"
 				(path "/59986deb-8fca-4720-9445-aa41ddfde149"
-					(reference "FUSE")
+					(reference "F1")
 					(unit 1)
 				)
@@
 		(dnp no)
 		(fields_autoplaced yes)
-		(property "Reference" "A"
+		(property "Reference" "J30"
 			(at 398.78 589.28 0)
 			(show_name no)
@@
 			)
 		)
-		(property "Value" "wire"
+		(property "Value" "A"
 			(at 398.78 591.82 0)
 			(show_name no)
@@
 			(project "main_pcb"
 				(path "/59986deb-8fca-4720-9445-aa41ddfde149"
-					(reference "A")
+					(reference "J30")
 					(unit 1)
 				)
@@
 		(dnp no)
 		(fields_autoplaced yes)
-		(property "Reference" "TREB_POS"
+		(property "Reference" "EXT5"
 			(at 721.36 636.2699 0)
 			(show_name no)
@@
 			)
 		)
-		(property "Value" "Conn_01x01"
+		(property "Value" "TREB_POS"
 			(at 721.36 638.8099 0)
 			(show_name no)
@@
 			(project "main_pcb"
 				(path "/59986deb-8fca-4720-9445-aa41ddfde149"
-					(reference "TREB_POS")
+					(reference "EXT5")
 					(unit 1)
 				)
@@
 		(dnp no)
 		(fields_autoplaced yes)
-		(property "Reference" "J?"
+		(property "Reference" "EXT2"
 			(at 887.73 877.5699 0)
 			(show_name no)
@@
 			(project "main_pcb"
 				(path "/59986deb-8fca-4720-9445-aa41ddfde149"
-					(reference "J?")
+					(reference "EXT2")
 					(unit 1)
 				)
