File: advent-powered-speaker/main_pcb_cleaned_up/main_pcb_cleaned_up.kicad_sch (KiCad schematic)
At the start: 151 parts, among them J1 wire, J10 wire, J11 wire, J12 wire, J13 wire, J14 wire, J15 wire, J16 wire, J17 wire, J18 wire, J20 wire, J21 wire, J22 wire, J30 A, J8 wire, J9 wire, Q1 C546B, Q10 C546B, Q11 C546B, Q12 C556B, Q13 C33740, Q14 C556B, Q15 KSE3055T, Q16 KSE3055T, Q17 KSE3055T, Q18 C33740, Q2 C32740, Q3 KSE3055T, Q4 C546(8)B, Q5 C32740, Q6 C546B, Q7 C546B, Q8 C556B, Q9 C556B, U1 4558DD JRC 4117B, U2 45560 JRC 4032A

Commit message: removed jumpers
Parts:
- removed J1, J10, J11, J12, J13, J14, J15, J16, J17, J18, J20, J21, J22, J8, J9: wire, symbol Jumper:Jumper_2_Bridged
- removed J30: A, symbol Jumper:Jumper_2_Bridged
Connections:
- net at C12.2, EXT1.5 (Pin_5), Q10.3 (Pin_3)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: now also C16.2, C2.2, C21.2, C24.2, C25.2, C27.2, C29.2, C6.1, C7.2, C9.2, D1.2 (-), D7.2 (A), EXT1.3 (Pin_3), EXT1.4 (Pin_4), EXT2.1 (Pin_1), H1.1, Q7.3 (Pin_3), R13.1, R14.2, R35.2, R41.1, R47.1, R51.1, R52.1, R55.2, R56.1, R57.1, R63.2, R66.1, R68.1, U1.4 (Pin_4), U2.4 (Pin_4)
- net at C27.1, R26.1, R47.2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: now also C26.2, R7.1
- net at C11.1, Q9.3 (Pin_3), R17.2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: now also Q1.3 (Pin_3), R48.1
- net at C23.1, C28.2, U2.2 (Pin_2): now also R61.2
- net at C2.1, D1.1 (+), R6.1: now also C29.1, EXT1.1 (Pin_1), EXT1.2 (Pin_2), Q1.1 (Pin_1), R3.1, R53.1, R54.2, R65.1
- net at F1.2: now also D1.3

Commit message: Added power rail symbols
Parts:
- removed U1: 4558DD JRC 4117B, symbol Connector_Generic:Conn_02x04_Counter_Clockwise
- removed U2: 45560 JRC 4032A, symbol Connector_Generic:Conn_02x04_Counter_Clockwise
- added U1: 4558DD JRC 4117B, Package_DIP:DIP-8_W7.62mm, symbol Amplifier_Operational:Opamp_Dual
- added U2: 4556D JRC 4032A, Package_DIP:DIP-8_W7.62mm, symbol Amplifier_Operational:Opamp_Dual
Connections:
- net -VDC: now reaches C12.2, C16.2, C2.2, C21.2, C24.2, C25.2, C27.2, C29.2, C6.1, C7.2, C9.2, D1.2 (-), D7.2 (A), EXT1.3 (Pin_3), EXT1.4 (Pin_4), EXT1.5 (Pin_5), EXT2.1 (Pin_1), H1.1, Q10.3 (Pin_3), Q11.3 (Pin_3), Q7.3 (Pin_3), R13.1, R14.2, R21.1, R25.1, R41.1, R47.1, R52.1, R55.2, R56.1, R57.1, R63.2, R66.1, R68.1
- net -VDC: now also R35.1, R51.2, U1.4 (V-), U2.4 (V-); no longer R35.2, R51.1
- net at C26.2, C27.1, R26.1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: now also U2.3 (+)
- net at C30.1, R67.2: now also U2.5 (+)
- net at R46.2, R60.1: now also U2.6 (-)
- net at D12.1 (K), Q12.2 (Pin_2): now also R35.2; no longer R35.1
- net at R5.2: now also U2.1
- net at C23.1, C28.2, R61.2: now also U2.2 (-)
- net at R2.1: now also D3.2 (A), Q4.2 (Pin_2), R34.1
- net OP_AMP_VDC: now reaches C11.1, Q1.3 (Pin_3), Q9.3 (Pin_3), R17.2, R19.2, R22.1, R48.1
- net OP_AMP_VDC: now also U1.8 (V+), U2.8 (V+)
- net at C8.1, R68.2, R7.2: now also U1.3 (+)
- net AUDIO_INPUT_TIP: now reaches EXT1.6 (Pin_6), R24.2, R49.2
- net +VDC: now reaches C2.1, C29.1, D1.1 (+), EXT1.1 (Pin_1), EXT1.2 (Pin_2), Q1.1 (Pin_1), R3.1, R53.1, R54.2, R6.1, R65.1
- net at R10.1, R12.2: now also U1.1
- net at R10.2, R11.2: now also U1.2 (-)
- net at C4.1, R26.2: now also U1.5 (+)
- net at R31.2, R33.1, R69.1: now also U1.6 (-)
- net at R1.2, R29.1, R32.2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: now also U1.7
- net at C17.2: now also C18.1; no longer C18.2
- new net: C18.2, R51.1
- new net: R2.2, U2.7
Other:
- note added: "NPN"
- note added: "PNP"
- moved on the sheet: C18, C2, C20, C24, C25, C29, C3, C7, D1, F1, H1, R2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
